File: boards/galvanika-board-1.0/galvanika-board-1.0.sch (EAGLE design)
At the start: 78 parts, among them IC1 LM358N, IC2 7805DT, IC3 74HC595D, IC4 74HC595D, IC5 74HC595D

Commit message: schema
Parts:
- added C10, C12, C8: 100n, rcl:C-EU025-025X050
- added C11: 47uF, rcl:CPOL-EUE2-4
- added C7, C9: 22p, rcl:C-EU025-025X050
- added IC6: ATMEGA48/88/168-PU, atmega8:ATMEGA48/88/168-PU
- added L1: 120mH, rcl:L-EU0207/10
- added Q1: 20MHz, crystal:CRYSTALHC49S
- added R47: 10K, rcl:R-EU_0207/10
- added R48: (no value), dragberry:R0904N
- added SA1, SA2: (no value), dragberry:SS12D00DIP
Connections:
- new net N$68: IC3A.SER, IC6.PB3(MOSI/OC2A/PCINT3)
- new net N$81: C7.2, IC6.PB6(XTAL1/TOSC1/PCINT6), Q1.2
- new net N$82: C9.2, IC6.PB7(XTAL2/TOSC2/PCINT7), Q1.1
- new net N$83: C10.1, IC6.AREF
- new net N$84: C12.1, IC6.AVCC, L1.2
- new net N$85: IC6.PC6(/RESET/PCINT14), R47.2
- new net N$86: IC3A.RCK, IC4A.RCK, IC5A.RCK, IC6.PB2(SS/OC1B/PCINT2)
- new net N$87: IC6.PB1(OC1A/PCINT1), SA1.O
- new net N$88: IC6.PC0(ADC0/PCINT8), R48.3
- new net N$89: IC6.PB0(ICP1/CLKO/PCINT0), SA1.S, SA2.P
- net +19V: now also SA2.O
- net GND: now also C10.2, C11.-, C12.2, C7.1, C8.2, C9.1, IC3A.G, IC4A.G, IC5A.G, IC6.AGND, IC6.GND@1, R48.1, SA2.S
- net N$11: now also IC6.PC1(ADC1/PCINT9)
- net N$25: now also SA1.P
- net N$28: now also IC6.PC2(ADC2/PCINT10)
- net N$35: now also IC6.PB5(SCK/PCINT5)
- net VCC: now also C11.+, C8.1, IC3A.SCL, IC4A.SCL, IC5A.SCL, IC6.VCC@1, L1.1, R47.1, R48.2

Commit message: board
Parts:
- added C13: 0.1uF, rcl:C-EU025-025X050
- added F1: 1.85A, dragberry:MF-R
- added JP1: (no value), pinhead:PINHD-1X6
- added R49: 10K, rcl:R-EU_R1206
- C1, C4: device rcl:C-EU050-025X075 -> rcl:C-EUC1206
- IC1: value LM358N -> LM358D; device linear:LM358N -> linear:LM358D
- IC3, IC4, IC5: value 74HC595D -> 74HCT595D; device 74xx-eu:74HC595D -> 74xx-eu:74HCT595D
- R12, R4, R5: device rcl:R-EU_0207/10 -> rcl:R-EU_R1206
Connections:
- net N$16 renamed A-RIGHT
- net N$17 renamed A-LEFT
- net N$18 renamed VO-RIGHT
- net N$24 renamed VI-RIGHT
- net N$5 renamed VI-LEFT
- net N$7 renamed VO-LEFT
- new net N$24: IC6.PB4(MISO/PCINT4), JP1.3
- new net N$90: R49.1, SA2.O
- new net N$91: F1.1, XS1.2
- net +19V: now also F1.2, R49.2; no longer SA2.O, XS1.2
- net GND: now also C13.2, JP1.6, R7.2; no longer R7.1
- net N$11: now also IC6.PC4(ADC4/SDA/PCINT12); no longer IC6.PC1(ADC1/PCINT9)
- net N$28: now also IC6.PC5(ADC5/SCLPCINT13); no longer IC6.PC2(ADC2/PCINT10)
- net N$35: now also JP1.2
- net N$46: no longer IC3A.QH*
- net N$68: now also JP1.4
- net N$85: now also JP1.1
- net N$89: now also C13.1
- net N$9: now also R7.1; no longer R7.2
- net VCC: now also JP1.5
Other:
- moved on the sheet: C5, C6, IC2, R7

Commit message: 'board'
Parts:
- added IC7: 74HC595D, 74xx-eu:74HC595D
- C13: device rcl:C-EU025-025X050 -> rcl:C-EUC1206
- C2, C3: device rcl:CPOL-EUE2.5-5 -> rcl:CPOL-EUE5-4
- R43, R44, R45, R46: device rcl:R-EU_R1206 -> rcl:R-EU_0207/7
- R49: device rcl:R-EU_R1206 -> rcl:R-EU_0207/10
Connections:
- net N$87 renamed PWM
- removed net N$50 (its old number): IC5A.QD, R28.2
- removed net N$65: IC3A.QF, R36.1
- removed net N$66: IC3A.QG, R37.1
- removed net N$67: IC3A.QH, R38.1
- removed net N$68: IC3A.SER, IC6.PB3(MOSI/OC2A/PCINT3), JP1.4
- removed net N$86: IC3A.RCK, IC4A.RCK, IC5A.RCK, IC6.PB2(SS/OC1B/PCINT2)
- removed net N$89: C13.1, IC6.PB0(ICP1/CLKO/PCINT0), SA1.S, SA2.P
- new net CLOCK: IC3A.SCK, IC4A.SCK, IC5A.SCK, IC6.PB5(SCK/PCINT5), IC7A.SCK, JP1.3
- new net DATA: IC3A.SER, IC6.PB3(MOSI/OC2A/PCINT3), JP1.1
- new net LATCH: IC3A.RCK, IC4A.RCK, IC5A.RCK, IC6.PB2(SS/OC1B/PCINT2), IC7A.RCK
- new net N$29: IC5A.QB, R22.1
- new net N$41: DZ1-7.A, R27.1
- new net N$55: IC3A.QG, R31.1
- new net PWM-CTRL: C13.1, IC6.PD1(TXD/PCINT17), SA1.S, SA2.P
- net +19V: no longer R49.2
- net GND: now also IC7A.G, R15.2, VT2.E, VT3.E, VT4.E; no longer R15.1
- net N$16: now also IC3A.QD, R38.1; no longer IC3A.QC, R33.1
- net N$17: now also IC3A.QC, R34.1; no longer IC3A.QA, R31.1
- net N$21: now also R15.1; no longer R15.2
- net N$24: now also JP1.2; no longer JP1.3
- net N$30: now also R22.2; no longer R23.1
- net N$31: now also IC5A.QC, R23.2; no longer DZ1-3.A, R25.1
- net N$32: now also DZ1-3.A, R23.1; no longer DZ1-4.A, R27.1
- net N$33: now also DZ1-4.A, R24.1; no longer DZ1-5.A, R29.1
- net N$34: now also IC5A.QD, R24.2; no longer IC5A.QF, R30.1
- net N$35: now also IC3A.QF, R37.1; no longer IC3A.SCK, IC4A.SCK, IC5A.SCK, IC6.PB5(SCK/PCINT5), JP1.2
- net N$36: now also IC5A.QE, R25.2; no longer IC4A.QE, R21.1
- net N$37: now also DZ1-5.A, R25.1; no longer DZ1-6.A, R22.2
- net N$38: now also IC5A.QF, R26.2; no longer DZ1-7.A, R24.1
- net N$39: now also DZ1-6.A; no longer DZ1-8.A
- net N$4: now also IC5A.QA, R21.1; no longer VT2.E, VT3.E, VT4.E
- net N$40: now also IC5A.QG, R27.2; no longer DZ1-9.A, R28.1
- net N$42: now also IC5A.QH, R28.2; no longer IC4A.QF, R22.1
- net N$43: now also DZ1-8.A, R28.1; no longer IC4A.QG, R23.2
- net N$44: now also IC3A.QH, R36.1; no longer IC4A.QH, R24.2
- net N$47: now also IC5A.QH*, IC7A.SER; no longer IC5A.QA, R25.2
- net N$48: now also IC7A.QA, R29.2; no longer IC5A.QB, R26.2
- net N$49: now also IC7A.QB, R30.1; no longer IC5A.QC, R27.2
- net N$51: now also DZ1-9.A, R29.1; no longer IC5A.QE, R29.2
- net N$61: now also IC3A.QA; no longer IC3A.QB
- net N$64: now also IC3A.QB; no longer IC3A.QE
- net N$7: now also IC3A.QE, R33.1; no longer IC3A.QD, R34.1
- net N$73: now also R41.2; no longer R39.2
- net N$75: now also R39.2; no longer R41.2
- net N$85: now also JP1.4; no longer JP1.1
- net VCC: now also IC7A.SCL, R49.2
Other:
- moved on the sheet: DZ1-1, DZ1-10, DZ1-2, DZ1-3, DZ1-4, DZ1-5, DZ1-6, DZ1-7, DZ1-8, DZ1-9, R15, R21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

Commit message: 'board'
Parts:
- C5: device rcl:C-EU050-025X075 -> rcl:C-EU025-025X050
Changed lines of the file:
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@@
 <part name="R20" library="rcl" library_urn="urn:adsk.eagle:library:334" deviceset="R-EU_" device="R1206" package3d_urn="urn:adsk.eagle:package:23540/2" value="100K"/>
 <part name="IC2" library="linear" library_urn="urn:adsk.eagle:library:262" deviceset="78*" device="DT" package3d_urn="urn:adsk.eagle:package:16415/2" technology="05"/>
-<part name="C5" library="rcl" deviceset="C-EU" device="050-025X075" package3d_urn="urn:adsk.eagle:package:23637/1" value="2.2uF"/>
+<part name="C5" library="rcl" deviceset="C-EU" device="025-025X050" package3d_urn="urn:adsk.eagle:package:23629/2" value="2.2uF"/>
 <part name="C6" library="rcl" library_urn="urn:adsk.eagle:library:334" deviceset="CPOL-EU" device="E2.5-5" package3d_urn="urn:adsk.eagle:package:23344/1" value="0.1uF"/>
 <part name="P+3" library="supply1" library_urn="urn:adsk.eagle:library:371" deviceset="VCC" device=""/>

Commit message: new board version
Parts:
- removed D1, D2: 1N5400, diode:1N5400
- removed IC2: 7805DT, linear:7805DT
- removed XS1: KLS2-2, dragberry:KLS2-2
- added D3, D4: 1N4001, tango:1N4001
- added J1: (no value), con-jack:DCJ0303
- added SA3, SA4: (no value), dragberry:SS12D00DIP
- added SA5: KCD11-101-H, dragberry:KCD11-101-H
- added U$3: L7805, dragberry:L7805
- R12, R5: value 2K -> (none); device rcl:R-EU_R1206 -> rcl:R-EU_0207/10
- R15, R7: value 10K -> (none); device dragberry:R0904N -> pot:3RP/1610N
- R21, R22, R23, R24, R25, R26, R31, R32, R33, R34, R35, R36, R37, R38: value (none) -> 330
- R39, R40, R41, R42: value (none) -> 200
- R4: value 200 -> (none); device rcl:R-EU_R1206 -> rcl:R-EU_0207/10
- R43, R44, R45, R46: device rcl:R-EU_0207/7 -> rcl:R-EU_R1206
- VT6, VT7: value BD139 -> IRF1404; device dragberry:BD139 -> dragberry:IRF1404
Connections:
- net N$25 renamed BRANCH-CTRL
- net N$90 renamed RIGHT-EN
- removed net N$46: IC4A.SER
- removed net N$55: IC3A.QG, R31.1
- removed net N$91: F1.1, XS1.2
- new net N$60: D4.CATHODE, VT7.S, XS2.1
- new net N$62: F1.1, J1.1
- new net N$63: SA3.S, SA4.S, XS2.2
- new net N$65: F1.2, SA5.P
- new net N$66: IC4A.SER, IC6.PB3(MOSI/OC2A/PCINT3), JP1.1
- new net N$67: IC3A.QG, R34.1
- net +19V: now also SA5.S, U$3.IN; no longer F1.2, IC2.VI
- net A-LEFT: now also VT7.D; no longer VT7.E
- net A-RIGHT: now also VT6.D; no longer VT6.E
- net DATA: now also IC4A.QH*; no longer IC6.PB3(MOSI/OC2A/PCINT3), JP1.1
- net GND: now also J1.3, R15.A, R7.A, U$3.GND; no longer IC2.GND, R15.2, R7.2, XS1.1
- net N$10: now also R7.S; no longer R7.3
- net N$12: now also R8.1, VT6.G; no longer R6.2, VT7.B
- net N$13: now also D3.CATHODE, VT6.S; no longer D1.C, VT6.C
- net N$14: now also R16G$1.2, SA3.P; no longer D2.C, VT7.C, XS2.1
- net N$15: now also R6.2, VT7.G; no longer R8.1, VT6.B
- net N$16: now also IC3A.QB, R31.1; no longer IC3A.QD, R38.1
- net N$17: now also IC3A.QH, R35.1; no longer IC3A.QC, R34.1
- net N$21: now also R15.E; no longer R15.1
- net N$23: now also R15.S; no longer R15.3
- net N$3: now also SA4.P; no longer R16G$1.2, XS2.2
- net N$35: now also R38.1; no longer R37.1
- net N$44: now also IC3A.QC; no longer IC3A.QH
- net N$45: now also IC3A.QH*; no longer IC4A.QH*
- net N$64: now also IC3A.QD, R37.1; no longer IC3A.QB, R35.1
- net N$9: now also R7.E; no longer R7.1
- net VCC: now also U$3.OUT; no longer IC2.VO
- net VO-LEFT: now also D3.ANODE; no longer D1.A
- net VO-RIGHT: now also D4.ANODE; no longer D2.A
Other:
- moved on the sheet: C3, C4, C5, C6, DA2, HG1, IC1A, LED2, R11, R12, R13, R14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

Commit message: 'board'
Parts:
- added C14: (no value), rcl:C-EUC1206
- added LED3, LED4: (no value), led:LED3MM
- added R50, R51, R52, R53: (no value), rcl:R-EU_R1206
- added SA6: KLS7-6X6, dragberry:KLS7-6X6
Connections:
- new net N$25: IC7A.QG, R50.2
- new net N$46: IC7A.QH, R51.1
- new net N$55: LED3.A, R50.1
- new net N$68: LED4.A, R51.2
- new net N$86: C14.1, IC6.PD2(INT0/PCINT18), R52.2, SA6.1
- new net N$87: R48.1, R53.2
- net A-LEFT: now also VT7.S; no longer VT7.D
- net A-RIGHT: now also VT6.S; no longer VT6.D
- net GND: now also C14.2, LED3.C, LED4.C, R53.1, SA6.2; no longer R48.1
- net N$13: now also VT6.D; no longer VT6.S
- net N$60: now also VT7.D, XS2.2; no longer VT7.S, XS2.1
- net N$63: now also XS2.1; no longer XS2.2
- net VCC: now also R52.1

Commit message: board
Parts:
- R1, R2: value 20K -> 100K
- R11: value 200 -> 240
- R13: value 20K -> 100k
- R14: value 20K -> 10k
- R15, R7: value (none) -> 2k
- R3: value 2k -> 10k
- R4: value (none) -> 240
Changed lines of the file:
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@@
 </classes>
 <parts>
-<part name="R1" library="rcl" library_urn="urn:adsk.eagle:library:334" deviceset="R-EU_" device="0207/10" package3d_urn="urn:adsk.eagle:package:23491/2" value="20K"/>
-<part name="R2" library="rcl" library_urn="urn:adsk.eagle:library:334" deviceset="R-EU_" device="0207/10" package3d_urn="urn:adsk.eagle:package:23491/2" value="20K"/>
-<part name="R3" library="rcl" library_urn="urn:adsk.eagle:library:334" deviceset="R-EU_" device="0207/10" package3d_urn="urn:adsk.eagle:package:23491/2" value="2k"/>
+<part name="R1" library="rcl" library_urn="urn:adsk.eagle:library:334" deviceset="R-EU_" device="0207/10" package3d_urn="urn:adsk.eagle:package:23491/2" value="100K"/>
+<part name="R2" library="rcl" library_urn="urn:adsk.eagle:library:334" deviceset="R-EU_" device="0207/10" package3d_urn="urn:adsk.eagle:package:23491/2" value="100K"/>
+<part name="R3" library="rcl" library_urn="urn:adsk.eagle:library:334" deviceset="R-EU_" device="0207/10" package3d_urn="urn:adsk.eagle:package:23491/2" value="10k"/>
 <part name="C1" library="rcl" library_urn="urn:adsk.eagle:library:334" deviceset="C-EU" device="C1206" package3d_urn="urn:adsk.eagle:package:23618/2" value="0.1uF"/>
 <part name="LED1" library="led" library_urn="urn:adsk.eagle:library:259" deviceset="LED" device="3MM" package3d_urn="urn:adsk.eagle:package:15797/1"/>
@@
 <part name="R10" library="rcl" library_urn="urn:adsk.eagle:library:334" deviceset="R-EU_" device="0411/12" package3d_urn="urn:adsk.eagle:package:23578/1" value="0.1"/>
 <part name="C3" library="rcl" deviceset="CPOL-EU" device="E5-4" package3d_urn="urn:adsk.eagle:package:23370/1" value="1uF"/>
-<part name="R11" library="rcl" library_urn="urn:adsk.eagle:library:334" deviceset="R-EU_" device="0207/10" package3d_urn="urn:adsk.eagle:package:23491/2" value="200"/>
+<part name="R11" library="rcl" library_urn="urn:adsk.eagle:library:334" deviceset="R-EU_" device="0207/10" package3d_urn="urn:adsk.eagle:package:23491/2" value="240"/>
 <part name="LED2" library="led" library_urn="urn:adsk.eagle:library:259" deviceset="LED" device="3MM" package3d_urn="urn:adsk.eagle:package:15797/1"/>
 <part name="C4" library="rcl" library_urn="urn:adsk.eagle:library:334" deviceset="C-EU" device="C1206" package3d_urn="urn:adsk.eagle:package:23618/2" value="0.1uF"/>
-<part name="R13" library="rcl" library_urn="urn:adsk.eagle:library:334" deviceset="R-EU_" device="0207/10" package3d_urn="urn:adsk.eagle:package:23491/2" value="20K"/>
-<part name="R14" library="rcl" library_urn="urn:adsk.eagle:library:334" deviceset="R-EU_" device="0207/10" package3d_urn="urn:adsk.eagle:package:23491/2" value="20K"/>
+<part name="R13" library="rcl" library_urn="urn:adsk.eagle:library:334" deviceset="R-EU_" device="0207/10" package3d_urn="urn:adsk.eagle:package:23491/2" value="100k"/>
+<part name="R14" library="rcl" library_urn="urn:adsk.eagle:library:334" deviceset="R-EU_" device="0207/10" package3d_urn="urn:adsk.eagle:package:23491/2" value="10k"/>
 <part name="GND1" library="supply1" library_urn="urn:adsk.eagle:library:371" deviceset="GND" device=""/>
 <part name="GND2" library="supply1" library_urn="urn:adsk.eagle:library:371" deviceset="GND" device=""/>
@@
 <part name="VT7" library="dragberry" deviceset="IRF1404" device="" package3d_urn="urn:adsk.eagle:package:29490/1"/>
 <part name="R5" library="rcl" deviceset="R-EU_" device="0207/10" package3d_urn="urn:adsk.eagle:package:23491/2"/>
-<part name="R7" library="pot" library_urn="urn:adsk.eagle:library:331" deviceset="3RP/1610N" device="" package3d_urn="urn:adsk.eagle:package:22726/1"/>
-<part name="R15" library="pot" library_urn="urn:adsk.eagle:library:331" deviceset="3RP/1610N" device="" package3d_urn="urn:adsk.eagle:package:22726/1"/>
+<part name="R7" library="pot" library_urn="urn:adsk.eagle:library:331" deviceset="3RP/1610N" device="" package3d_urn="urn:adsk.eagle:package:22726/1" value="2k"/>
+<part name="R15" library="pot" library_urn="urn:adsk.eagle:library:331" deviceset="3RP/1610N" device="" package3d_urn="urn:adsk.eagle:package:22726/1" value="2k"/>
 <part name="SA5" library="dragberry" deviceset="KCD11-101-H" device=""/>
 <part name="R46" library="rcl" deviceset="R-EU_" device="R1206" package3d_urn="urn:adsk.eagle:package:23540/2"/>
@@
 <part name="SA3" library="dragberry" deviceset="SS12D00" device="DIP"/>
 <part name="SA4" library="dragberry" deviceset="SS12D00" device="DIP"/>
-<part name="R4" library="rcl" deviceset="R-EU_" device="0207/10" package3d_urn="urn:adsk.eagle:package:23491/2"/>
+<part name="R4" library="rcl" deviceset="R-EU_" device="0207/10" package3d_urn="urn:adsk.eagle:package:23491/2" value="240"/>
 <part name="C5" library="rcl" deviceset="C-EU" device="025-025X050" package3d_urn="urn:adsk.eagle:package:23629/2" value="2.2uF"/>
 <part name="R50" library="rcl" library_urn="urn:adsk.eagle:library:334" deviceset="R-EU_" device="R1206" package3d_urn="urn:adsk.eagle:package:23540/2"/>
@@
 </instance>
 <instance part="R15" gate="G$1" x="147.32" y="20.32" smashed="yes">
-<attribute name="NAME" x="143.891" y="16.51" size="1.778" layer="95" rot="R90"/>
-<attribute name="VALUE" x="143.51" y="16.51" size="1.778" layer="96" rot="R90"/>
+<attribute name="NAME" x="143.891" y="19.05" size="1.778" layer="95" rot="R90"/>
+<attribute name="VALUE" x="151.13" y="16.51" size="1.778" layer="96" rot="R90"/>
 </instance>
 <instance part="SA5" gate="G$1" x="40.64" y="119.38" smashed="yes" rot="R270">
