File: boards/galvanika-board-1.0/galvanika-board-1.0.sch (EAGLE design)
At the start: 107 parts, among them IC1 LM358D, IC3 74HCT595D, IC4 74HCT595D, IC5 74HCT595D, IC6 ATMEGA48/88/168-PU, IC7 74HC595D, Q1 20MHz

Commit message: program
Connections:
- net N$24 renamed MISO
- net N$66 renamed MOSI
Changed lines of the file:
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@@
 </segment>
 </net>
-<net name="N$24" class="0">
+<net name="MISO" class="0">
 <segment>
 <pinref part="IC6" gate="1" pin="PB4(MISO/PCINT4)"/>
@@
 </segment>
 </net>
-<net name="N$66" class="0">
+<net name="MOSI" class="0">
 <segment>
 <pinref part="IC6" gate="1" pin="PB3(MOSI/OC2A/PCINT3)"/>
