File: boards/galvanika-board-1.0/galvanika-board-1.0.sch (EAGLE design)
At the start: 107 parts, among them IC1 LM358D, IC3 74HCT595D, IC4 74HCT595D, IC5 74HCT595D, IC6 ATMEGA48/88/168-PU, IC7 74HC595D, Q1 20MHz

Commit message: board v1
Parts:
- added R54, R55: 100k, rcl:R-EU_R1206
Connections:
- net GND: now also R54.1, R55.1
- net N$12: now also R54.2
- net N$15: now also R55.2
Changed lines of the file:
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@@
 <part name="GND4" library="supply1" library_urn="urn:adsk.eagle:library:371" deviceset="GND" device=""/>
 <part name="R53" library="rcl" deviceset="R-EU_" device="R1206" package3d_urn="urn:adsk.eagle:package:23540/2"/>
+<part name="R54" library="rcl" deviceset="R-EU_" device="R1206" package3d_urn="urn:adsk.eagle:package:23540/2" value="100k"/>
+<part name="R55" library="rcl" deviceset="R-EU_" device="R1206" package3d_urn="urn:adsk.eagle:package:23540/2" value="100k"/>
 </parts>
 <sheets>
@@
 <attribute name="NAME" x="-148.8186" y="123.19" size="1.778" layer="95" rot="R90"/>
 <attribute name="VALUE" x="-144.018" y="123.19" size="1.778" layer="96" rot="R90"/>
+</instance>
+<instance part="R54" gate="G$1" x="96.52" y="-7.62" smashed="yes" rot="R90">
+<attribute name="NAME" x="95.0214" y="-11.43" size="1.778" layer="95" rot="R90"/>
+<attribute name="VALUE" x="99.822" y="-11.43" size="1.778" layer="96" rot="R90"/>
+</instance>
+<instance part="R55" gate="G$1" x="114.3" y="-7.62" smashed="yes" rot="R90">
+<attribute name="NAME" x="112.8014" y="-11.43" size="1.778" layer="95" rot="R90"/>
+<attribute name="VALUE" x="117.602" y="-11.43" size="1.778" layer="96" rot="R90"/>
 </instance>
 </instances>
@@
 <junction x="71.12" y="-15.24"/>
 <pinref part="R9" gate="G$1" pin="1"/>
-<wire x1="124.46" y1="-15.24" x2="104.14" y2="-15.24" width="0.1524" layer="91"/>
+<wire x1="124.46" y1="-15.24" x2="114.3" y2="-15.24" width="0.1524" layer="91"/>
 <junction x="86.36" y="-15.24"/>
 <pinref part="C3" gate="G$1" pin="-"/>
-<wire x1="104.14" y1="-15.24" x2="86.36" y2="-15.24" width="0.1524" layer="91"/>
+<wire x1="114.3" y1="-15.24" x2="104.14" y2="-15.24" width="0.1524" layer="91"/>
+<wire x1="104.14" y1="-15.24" x2="96.52" y2="-15.24" width="0.1524" layer="91"/>
+<wire x1="96.52" y1="-15.24" x2="86.36" y2="-15.24" width="0.1524" layer="91"/>
 <wire x1="139.7" y1="30.48" x2="139.7" y2="-15.24" width="0.1524" layer="91"/>
 <wire x1="139.7" y1="-15.24" x2="124.46" y2="-15.24" width="0.1524" layer="91"/>
@@
 <wire x1="-22.86" y1="-5.08" x2="-22.86" y2="-2.54" width="0.1524" layer="91"/>
 <junction x="-22.86" y="-2.54"/>
+<pinref part="R54" gate="G$1" pin="1"/>
+<wire x1="96.52" y1="-12.7" x2="96.52" y2="-15.24" width="0.1524" layer="91"/>
+<junction x="96.52" y="-15.24"/>
+<pinref part="R55" gate="G$1" pin="1"/>
+<wire x1="114.3" y1="-12.7" x2="114.3" y2="-15.24" width="0.1524" layer="91"/>
+<junction x="114.3" y="-15.24"/>
 </segment>
 <segment>
@@
 <segment>
 <pinref part="R8" gate="G$1" pin="1"/>
-<wire x1="93.98" y1="10.16" x2="101.6" y2="10.16" width="0.1524" layer="91"/>
+<wire x1="93.98" y1="10.16" x2="96.52" y2="10.16" width="0.1524" layer="91"/>
 <pinref part="VT6" gate="G$1" pin="G"/>
+<pinref part="R54" gate="G$1" pin="2"/>
+<wire x1="96.52" y1="10.16" x2="101.6" y2="10.16" width="0.1524" layer="91"/>
+<wire x1="96.52" y1="-2.54" x2="96.52" y2="10.16" width="0.1524" layer="91"/>
+<junction x="96.52" y="10.16"/>
 </segment>
 </net>
@@
 <segment>
 <pinref part="R6" gate="G$1" pin="2"/>
-<wire x1="111.76" y1="0" x2="116.84" y2="0" width="0.1524" layer="91"/>
+<wire x1="111.76" y1="0" x2="114.3" y2="0" width="0.1524" layer="91"/>
 <pinref part="VT7" gate="G$1" pin="G"/>
-</segment>
-</net>
+<pinref part="R55" gate="G$1" pin="2"/>
+<wire x1="114.3" y1="0" x2="116.84" y2="0" width="0.1524" layer="91"/>
+<wire x1="114.3" y1="-2.54" x2="114.3" y2="0" width="0.1524" layer="91"/>
+<junction x="114.3" y="0"/>
+</segment>
+</net>
