File: boards/galvanika-board-1.0/galvanika-board-1.0.brd (EAGLE design)
At the start: 100 x 50 mm, 78 parts, among them IC1 LM358N, IC2 7805DT, IC3 74HC595D, IC4 74HC595D, IC5 74HC595D

Commit message: schema
Parts:
- added C10, C12, C8: 100n, rcl:C025-025X050
- added C11: 47uF, rcl:E2-4
- added C7, C9: 22p, rcl:C025-025X050
- added IC6: ATMEGA48/88/168-PU, atmega8:DIL28-3
- added L1: 120mH, rcl:0207/10
- added Q1: 20MHz, crystal:HC49/S
- added R47: 10K, rcl:0207/10
- added R48: (no value), dragberry:R0904N
- added SA1, SA2: (no value), dragberry:SS12D00
- moved DA2 4.40 mm to (15.7, 42.7)
Connections:
- new net N$68: IC3.14, IC6.17
- new net N$81: C7.2, IC6.9, Q1.2
- new net N$82: C9.2, IC6.10, Q1.1
- new net N$83: C10.1, IC6.21
- new net N$84: C12.1, IC6.20, L1.2
- new net N$85: IC6.1, R47.2
- new net N$86: IC3.12, IC4.12, IC5.12, IC6.16
- new net N$87: IC6.15, SA1.1$O
- new net N$88: IC6.23, R48.2
- new net N$89: IC6.14, SA1.1$S, SA2.1$P
- net +19V: now also SA2.1$O
- net GND: now also C10.2, C11.-, C12.2, C7.1, C8.2, C9.1, IC3.13, IC4.13, IC5.13, IC6.22, IC6.8, R48.1, SA2.1$S
- net N$11: now also IC6.24
- net N$25: now also SA1.1$P
- net N$28: now also IC6.25
- net N$35: now also IC6.19
- net VCC: now also C11.+, C8.1, IC3.10, IC4.10, IC5.10, IC6.7, L1.1, R47.1, R48.3
Other:
- board size 100 x 50 mm -> 100 x 80 mm

Commit message: board
Parts:
- added C13: 0.1uF, rcl:C025-025X050
- added F1: 1.85A, dragberry:MF-R
- added JP1: (no value), pinhead:1X06
- added R49: 10K, rcl:R1206
- C1, C4: device rcl:C050-025X075 -> rcl:C1206
- IC1: value LM358N -> LM358D; device linear:DIL08 -> linear:SO08
- IC3, IC4, IC5: value 74HC595D -> 74HCT595D
- R12, R4, R5: device rcl:0207/10 -> rcl:R1206
- moved R47 576.6 mm to (38.5, 44.2)
- moved SA2 560.3 mm to (56.7, 17.2)
- moved C11 551.1 mm to (40.6, 30.3), turned to 270 degrees
- moved L1 550.2 mm to (35.1, 22.6), turned to 270 degrees
- moved C8 549.5 mm to (40.6, 34.0), turned to 180 degrees
- moved C12 547.2 mm to (57.2, 22.0), turned to 270 degrees
- moved C10 543.7 mm to (57.2, 27.1), turned to 90 degrees
- moved SA1 539.0 mm to (36.8, 3.00)
- moved R45 536.7 mm to (85.8, 41.2), flipped to the bottom
- moved Q1 529.6 mm to (40.6, 22.1), turned to 90 degrees
- moved C9 526.8 mm to (40.5, 11.9), turned to 180 degrees
- moved R41 523.5 mm to (85.8, 44.4), flipped to the bottom, turned to 180 degrees
- moved C7 520.0 mm to (40.5, 14.9), turned to 180 degrees
- moved R40 515.0 mm to (64.2, 45.1), flipped to the bottom, turned to 180 degrees
- moved R39 507.5 mm to (64.5, 41.6), flipped to the bottom, turned to 180 degrees
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Connections:
- net N$16 renamed A-RIGHT
- net N$17 renamed A-LEFT
- net N$18 renamed VO-RIGHT
- net N$24 renamed VI-RIGHT
- net N$5 renamed VI-LEFT
- net N$7 renamed VO-LEFT
- new net N$24: IC6.18, JP1.3
- new net N$90: R49.1, SA2.1$O
- new net N$91: F1.1, XS1.2
- net +19V: now also F1.2, R49.2; no longer IC3.16, IC4.16, IC5.16, SA2.1$O, XS1.2
- net GND: now also C13.2, JP1.6, R7.3; no longer R7.1
- net N$11: now also IC6.27; no longer IC6.24
- net N$28: now also IC6.28; no longer IC6.25
- net N$35: now also JP1.2
- net N$46: no longer IC3.9
- net N$68: now also JP1.4
- net N$85: now also JP1.1
- net N$89: now also C13.1
- net N$9: now also R7.1; no longer R7.3
- net VCC: now also IC3.16, IC4.16, IC5.16, JP1.5
Routing:
- net GND: track 0.00 -> 303.7 mm, vias 0 -> 6
- net +19V: track 0.00 -> 119.6 mm
- net N$13: track 0.00 -> 101.7 mm
- net N$10: track 0.00 -> 79.9 mm
- net VO-LEFT: track 0.00 -> 75.0 mm
- net VI-LEFT: track 0.00 -> 60.4 mm
- net VI-RIGHT: track 0.00 -> 58.4 mm
- net N$15: track 0.00 -> 51.4 mm
- net N$14: track 0.00 -> 50.7 mm
- net N$12: track 0.00 -> 44.7 mm
- net A-RIGHT: track 0.00 -> 44.1 mm
- net A-LEFT: track 0.00 -> 43.1 mm
- net N$3: track 0.00 -> 31.6 mm
- net N$28: track 0.00 -> 19.4 mm, vias 0 -> 2
- net N$11: track 0.00 -> 19.3 mm
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
Commit message: 'board'
Parts:
- added IC7: 74HC595D, 74xx-eu:SO16
- C13: device rcl:C025-025X050 -> rcl:C1206
- C2, C3: device rcl:E2,5-5 -> rcl:E5-4
- R43, R44, R45, R46: device rcl:R1206 -> rcl:0207/7
- R49: device rcl:R1206 -> rcl:0207/10
- moved IC4 61.4 mm to (64.4, 42.2)
- moved R14 60.1 mm to (11.0, 63.9)
- moved VT4 51.5 mm to (10.7, 68.5), turned to 180 degrees
- moved IC2 49.6 mm to (36.8, 54.3)
- moved R46 47.6 mm to (70.5, 56.1), flipped to the top, turned to 90 degrees
- moved R3 47.2 mm to (11.0, 57.8), turned to 180 degrees
- moved R44 43.2 mm to (81.6, 56.1), flipped to the top, turned to 90 degrees
- moved R49 41.4 mm to (78.2, 11.6), turned to 90 degrees
- moved C6 40.2 mm to (41.5, 48.0), turned to 180 degrees
- moved VT3 40.1 mm to (10.8, 52.8)
- moved JP1 39.6 mm to (69.7, 17.6)
- moved R43 39.5 mm to (76.1, 56.1), flipped to the top, turned to 90 degrees
- moved C13 38.4 mm to (32.9, 46.5), flipped to the bottom
- moved VT11 37.6 mm to (73.3, 49.5), turned to 270 degrees
- moved SA1 36.7 mm to (35.5, 39.7), turned to 90 degrees
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Connections:
- net N$87 renamed PWM
- removed net N$50 (its old number): IC5.3, R28.2
- removed net N$65: IC3.5, R36.1
- removed net N$66: IC3.6, R37.1
- removed net N$67: IC3.7, R38.1
- removed net N$68: IC3.14, IC6.17, JP1.4
- removed net N$86: IC3.12, IC4.12, IC5.12, IC6.16
- removed net N$89: C13.1, IC6.14, SA1.1$S, SA2.1$P
- new net CLOCK: IC3.11, IC4.11, IC5.11, IC6.19, IC7.11, JP1.3
- new net DATA: IC3.14, IC6.17, JP1.1
- new net LATCH: IC3.12, IC4.12, IC5.12, IC6.16, IC7.12
- new net N$29: IC5.1, R22.1
- new net N$41: DZ1.7, R27.1
- new net N$55: IC3.6, R31.1
- new net PWM-CTRL: C13.1, IC6.3, SA1.1$S, SA2.1$P
- net +19V: no longer R49.2
- net GND: now also IC7.13, IC7.8, R15.3, VT2.3, VT3.3, VT4.3; no longer R15.1
- net N$16: now also IC3.3, R38.1; no longer IC3.2, R33.1
- net N$17: now also IC3.2, R34.1; no longer IC3.15, R31.1
- net N$21: now also R15.1; no longer R15.3
- net N$24: now also JP1.2; no longer JP1.3
- net N$30: now also R22.2; no longer R23.1
- net N$31: now also IC5.2, R23.2; no longer DZ1.3, R25.1
- net N$32: now also DZ1.3, R23.1; no longer DZ1.4, R27.1
- net N$33: now also DZ1.4, R24.1; no longer DZ1.5, R29.1
- net N$34: now also IC5.3, R24.2; no longer IC5.5, R30.1
- net N$35: now also IC3.5, R37.1; no longer IC3.11, IC4.11, IC5.11, IC6.19, JP1.2
- net N$36: now also IC5.4, R25.2; no longer IC4.4, R21.1
- net N$37: now also DZ1.5, R25.1; no longer DZ1.6, R22.2
- net N$38: now also IC5.5, R26.2; no longer DZ1.7, R24.1
- net N$39: now also DZ1.6; no longer DZ1.8
- net N$4: now also IC5.15, R21.1; no longer VT2.3, VT3.3, VT4.3
- net N$40: now also IC5.6, R27.2; no longer DZ1.9, R28.1
- net N$42: now also IC5.7, R28.2; no longer IC4.5, R22.1
- net N$43: now also DZ1.8, R28.1; no longer IC4.6, R23.2
- net N$44: now also IC3.7, R36.1; no longer IC4.7, R24.2
- net N$47: now also IC5.9, IC7.14; no longer IC5.15, R25.2
- net N$48: now also IC7.15, R29.2; no longer IC5.1, R26.2
- net N$49: now also IC7.1, R30.1; no longer IC5.2, R27.2
- net N$51: now also DZ1.9, R29.1; no longer IC5.4, R29.2
- net N$61: now also IC3.15; no longer IC3.1
- net N$64: now also IC3.1; no longer IC3.4
- net N$7: now also IC3.4, R33.1; no longer IC3.3, R34.1
- net N$73: now also R41.2; no longer R39.2
- net N$75: now also R39.2; no longer R41.2
- net N$85: now also JP1.4; no longer JP1.1
- net VCC: now also IC7.10, IC7.16, R49.2
Routing:
- net GND: track 303.7 -> 745.0 mm, vias 6 -> 14
- net VCC: track 10.0 -> 378.4 mm, vias 0 -> 24
- net +19V: track 119.6 -> 313.9 mm, vias 0 -> 2
- net LATCH: track 0.00 -> 149.2 mm, vias 0 -> 4
- net CLOCK: track 0.00 -> 146.3 mm, vias 0 -> 6
- net N$20: track 0.00 -> 141.7 mm, vias 0 -> 4
- net PWM-CTRL: track 0.00 -> 110.3 mm, vias 0 -> 8
- net N$23: track 0.00 -> 100.6 mm, vias 0 -> 2
- net N$45: track 0.00 -> 90.0 mm, vias 0 -> 6
- net N$21: track 0.00 -> 81.4 mm
- net N$1: track 6.08 -> 78.4 mm, vias 0 -> 4
- net N$85: track 0.00 -> 69.7 mm, vias 0 -> 2
- net N$88: track 0.00 -> 63.8 mm, vias 0 -> 2
- net N$25: track 0.00 -> 61.2 mm
- net PWM: track 0.00 -> 39.8 mm, vias 0 -> 2
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- added copper zone on layer 16, net +19V
- added copper zone on layer 16, net VI-LEFT
- added copper zone on layer 16, net VI-RIGHT
Other:
- board size 100 x 80 mm -> 100 x 100 mm
- board text added: "DRAGBERRY"

Commit message: 'board'
Parts:
- C5: device rcl:C050-025X075 -> rcl:C025-025X050
- moved C5 22.6 mm to (42.7, 59.5)
- moved D1 2.10 mm to (78.5, 75.7)
- moved C2 1.35 mm to (85.2, 81.7), turned to 270 degrees
- moved R7 1.20 mm to (87.6, 6.70)
- moved R13 0.90 mm to (93.2, 68.5)
- moved R42 0.40 mm to (68.1, 50.0)
- moved R16 0.16 mm to (50.0, 78.3)
- moved R48 0.14 mm to (34.3, 7.90)
Routing:
- net PWM-CTRL: track 110.3 -> 118.7 mm
- net GND: track 745.0 -> 753.1 mm, vias 14 -> 16
- net +19V: track 313.9 -> 321.0 mm
- net VO-LEFT: track 97.4 -> 102.4 mm
- net N$13: track 103.0 -> 100.9 mm
- net N$80: track 25.5 -> 27.6 mm
- net N$21: track 81.4 -> 79.4 mm
- net N$23: track 100.6 -> 99.6 mm
- net N$10: track 103.6 -> 104.5 mm
- net N$20: track 141.7 -> 140.8 mm
- net A-RIGHT: track 44.6 -> 45.3 mm
- net VO-RIGHT: track 33.9 -> 34.6 mm
- added copper zone on layer 16, net N$91
Other:
- board text added: "GALVANIKA"

Commit message: new board version
Parts:
- removed D1, D2: 1N5400, diode:DO201-15
- removed IC2: 7805DT, linear:TO252
- removed XS1: KLS2-2, dragberry:KLS2-2
- added D3, D4: 1N4001, tango:DO41-10
- added J1: (no value), con-jack:DCJ0303
- added SA3, SA4: (no value), dragberry:SS12D00
- added SA5: KCD11-101-H, dragberry:KCD11-101-H
- added U$3: L7805, dragberry:TO220-SK29-38S
- R12, R5: value 2K -> (none); device rcl:R1206 -> rcl:0207/10
- R15, R7: value 10K -> (none); device dragberry:R0904N -> pot:3RP/1610N
- R21, R22, R23, R24, R25, R26, R31, R32, R33, R34, R35, R36, R37, R38: value (none) -> 330
- R39, R40, R41, R42: value (none) -> 200
- R4: value 200 -> (none); device rcl:R1206 -> rcl:0207/10
- R43, R44, R45, R46: device rcl:0207/7 -> rcl:R1206
- VT6, VT7: value BD139 -> IRF1404; device dragberry:TO126AV -> dragberry:TO220-V
- moved R4 105.9 mm to (109.5, 114.8), flipped to the top, turned to 90 degrees
- moved F1 100.6 mm to (19.0, 92.0), turned to 90 degrees
- moved R48 77.0 mm to (111.2, 7.25), turned to 270 degrees
- moved R7 76.0 mm to (121.0, 75.0), turned to 90 degrees
- moved SA2 68.4 mm to (24.5, 54.2), turned to 0 degrees
- moved R15 67.6 mm to (4.00, 75.0), turned to 270 degrees
- moved C5 67.2 mm to (6.00, 115.8), turned to 180 degrees
- moved C1 65.6 mm to (101.0, 145.0), turned to 90 degrees
- moved C3 61.4 mm to (37.0, 139.5), turned to 0 degrees
- moved C10 60.3 mm to (117.8, 40.2), turned to 180 degrees
- moved C12 60.1 mm to (117.8, 34.5), turned to 0 degrees
- moved C9 60.1 mm to (97.8, 41.5), turned to 180 degrees
- moved L1 58.4 mm to (108.5, 40.8)
- moved IC6 58.3 mm to (108.2, 39.2)
- moved C2 57.6 mm to (87.8, 139.2), turned to 180 degrees
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Connections:
- net N$25 renamed BRANCH-CTRL
- net N$90 renamed RIGHT-EN
- removed net N$46: IC4.14
- removed net N$55: IC3.6, R31.1
- removed net N$91: F1.1, XS1.2
- new net N$60: D4.C, VT7.S, XS2.1
- new net N$62: F1.1, J1.1
- new net N$63: SA3.1$S, SA4.1$S, XS2.2
- new net N$65: F1.2, SA5.2
- new net N$66: IC4.14, IC6.17, JP1.1
- new net N$67: IC3.6, R34.1
- net +19V: now also SA5.3, U$3.1; no longer F1.2, IC2.1
- net A-LEFT: now also VT7.D; no longer VT7.E
- net A-RIGHT: now also VT6.D; no longer VT6.E
- net DATA: now also IC4.9; no longer IC6.17, JP1.1
- net GND: now also J1.3, R15.1, R7.1, U$3.2; no longer IC2.3, R15.3, R7.3, XS1.1
- net N$12: now also R8.1, VT6.G; no longer R6.2, VT7.B
- net N$13: now also D3.C, VT6.S; no longer D1.C, VT6.C
- net N$14: now also R16.2, SA3.1$P; no longer D2.C, VT7.C, XS2.1
- net N$15: now also R6.2, VT7.G; no longer R8.1, VT6.B
- net N$16: now also IC3.1, R31.1; no longer IC3.3, R38.1
- net N$17: now also IC3.7, R35.1; no longer IC3.2, R34.1
- net N$21: now also R15.3; no longer R15.1
- net N$3: now also SA4.1$P; no longer R16.2, XS2.2
- net N$35: now also R38.1; no longer R37.1
- net N$44: now also IC3.2; no longer IC3.7
- net N$45: now also IC3.9; no longer IC4.9
- net N$64: now also IC3.3, R37.1; no longer IC3.1, R35.1
- net N$9: now also R7.3; no longer R7.1
- net VCC: now also U$3.3; no longer IC2.2
- net VO-LEFT: now also D3.A; no longer D1.A
- net VO-RIGHT: now also D4.A; no longer D2.A
Routing:
- net GND: track 753.1 -> 1309.8 mm, vias 16 -> 6
- net VCC: track 378.3 -> 592.4 mm, vias 24 -> 16
- net +19V: track 321.0 -> 210.7 mm, vias 2 -> 0
- net N$28: track 37.9 -> 138.5 mm, vias 2 -> 6
- net N$66: track 0.00 -> 88.9 mm
- net VI-LEFT: track 61.9 -> 147.4 mm
- net N$11: track 31.0 -> 109.5 mm, vias 0 -> 4
- net N$45: track 90.0 -> 22.3 mm, vias 6 -> 0
- net N$20: track 140.8 -> 73.9 mm, vias 4 -> 0
- net PWM: track 39.8 -> 100.0 mm, vias 2 -> 4
- net CLOCK: track 146.6 -> 200.2 mm, vias 6 -> 8
- net VO-LEFT: track 102.4 -> 61.5 mm
- net N$60: track 0.00 -> 36.0 mm
- net N$21: track 79.4 -> 44.0 mm
- net N$63: track 0.00 -> 35.0 mm
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- added copper zone on layer 16, net GND
- added copper zone on layer 16, net VCC
- removed copper zone on layer 16, net +19V
- removed copper zone on layer 16, net N$91
- removed copper zone on layer 16, net VI-LEFT
- removed copper zone on layer 16, net VI-RIGHT
Other:
- board size 100 x 100 mm -> 125.1 x 150 mm

Commit message: 'board'
Parts:
- added C14: (no value), rcl:C1206
- added LED3, LED4: (no value), led:LED3MM
- added R50, R51, R52, R53: (no value), rcl:R1206
- added SA6: KLS7-6X6, dragberry:KLS7-6X6
- moved R15 2.75 mm to (6.75, 75.0)
- moved R7 2.75 mm to (118.2, 75.0)
- moved VT6 2.00 mm to (84.0, 121.0)
- moved VT7 2.00 mm to (41.0, 121.0)
- moved VT3 1.75 mm to (35.8, 93.2)
- moved XS2 1.60 mm to (62.0, 142.5), turned to 180 degrees
- moved R12 0.75 mm to (18.8, 132.0)
- moved R17 0.75 mm to (70.2, 117.8)
- moved R20 0.75 mm to (53.8, 117.8)
- moved R8 0.75 mm to (18.8, 125.2)
- moved IC1 0.25 mm to (62.2, 121.0)
Connections:
- new net N$25: IC7.6, R50.2
- new net N$46: IC7.7, R51.1
- new net N$55: LED3.A, R50.1
- new net N$68: LED4.A, R51.2
- new net N$86: C14.1, IC6.4, R52.2, SA6.P$1, SA6.P$2
- new net N$87: R48.1, R53.2
- net A-LEFT: now also VT7.S; no longer VT7.D
- net A-RIGHT: now also VT6.S; no longer VT6.D
- net GND: now also C14.2, LED3.K, LED4.K, R53.1, SA6.P$3, SA6.P$4; no longer R48.1
- net N$13: now also VT6.D; no longer VT6.S
- net N$60: now also VT7.D, XS2.2; no longer VT7.S, XS2.1
- net N$63: now also XS2.1; no longer XS2.2
- net VCC: now also R52.1
Routing:
- net GND: track 1309.8 -> 1511.3 mm, vias 6 -> 4
- net N$86: track 0.00 -> 67.3 mm
- net VCC: track 592.4 -> 575.5 mm
- net N$20: track 73.9 -> 87.0 mm
- net BRANCH-CTRL: track 55.8 -> 66.6 mm
- net N$25: track 0.00 -> 10.4 mm
- net A-LEFT: track 40.3 -> 49.2 mm
- net +19V: track 210.7 -> 218.0 mm
- net N$46: track 0.00 -> 7.10 mm
- net N$3: track 15.2 -> 20.6 mm
- net A-RIGHT: track 30.9 -> 25.6 mm
- net N$87: track 0.00 -> 5.27 mm
- net N$60: track 36.0 -> 41.0 mm
- net N$2: track 27.2 -> 22.3 mm
- net N$15: track 47.0 -> 42.6 mm
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- added copper zone on layer 16, net VO-LEFT

Commit message: board
Parts:
- R1, R2: value 20K -> 100K
- R11: value 200 -> 240
- R13: value 20K -> 100k
- R14: value 20K -> 10k
- R15, R7: value (none) -> 2k
- R3: value 2k -> 10k
- R4: value (none) -> 240

Commit message: board
Parts:
- moved C5 61.9 mm to (59.8, 85.0)
- moved C2 4.10 mm to (85.2, 136.0)
- moved C3 3.55 mm to (39.2, 136.8)
- moved SA1 2.45 mm to (41.7, 56.5)
- moved SA2 0.60 mm to (24.5, 54.9)
- moved SA3 0.35 mm to (48.4, 143.0)
- moved SA4 0.20 mm to (77.8, 143.0)
Routing:
- net GND: track 1511.3 -> 1501.8 mm
- net PWM: track 100.0 -> 97.4 mm
- net BRANCH-CTRL: track 66.6 -> 69.0 mm
- net VI-LEFT: track 148.9 -> 150.9 mm
- net +19V: track 218.0 -> 216.5 mm
- net VO-LEFT: track 61.5 -> 62.8 mm
- net VO-RIGHT: track 67.4 -> 68.5 mm
- net N$26: track 18.5 -> 17.6 mm
- net PWM-CTRL: track 91.5 -> 90.8 mm
- net RIGHT-EN: track 38.6 -> 38.0 mm
- net N$63: track 34.8 -> 34.3 mm
Other:
- board text added: "CUPRUMBERRY"
- board text added: "DRAGBERRY 2020"
- board text removed: "DRAGBERRY"
