File: boards/galvanika-board-1.0/galvanika-board-1.0.brd (EAGLE design)
At the start: 125.1 x 150 mm, 107 parts, among them IC1 LM358D, IC3 74HCT595D, IC4 74HCT595D, IC5 74HCT595D, IC6 ATMEGA48/88/168-PU, IC7 74HC595D, Q1 20MHz

Commit message: program
Connections:
- net N$24 renamed MISO
- net N$66 renamed MOSI
Changed lines of the file:
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@@
 <grid distance="0.25" unitdist="mm" unit="mm" style="lines" multiple="1" display="yes" altdistance="5" altunitdist="mil" altunit="mil"/>
 <layers>
-<layer number="1" name="Top" color="4" fill="1" visible="no" active="yes"/>
+<layer number="1" name="Top" color="4" fill="1" visible="yes" active="yes"/>
 <layer number="2" name="Route2" color="16" fill="1" visible="no" active="no"/>
 <layer number="3" name="Route3" color="17" fill="1" visible="no" active="no"/>
@@
 <layer number="19" name="Unrouted" color="6" fill="1" visible="no" active="yes"/>
 <layer number="20" name="Dimension" color="24" fill="1" visible="yes" active="yes"/>
-<layer number="21" name="tPlace" color="7" fill="1" visible="no" active="yes"/>
-<layer number="22" name="bPlace" color="7" fill="1" visible="no" active="yes"/>
-<layer number="23" name="tOrigins" color="15" fill="1" visible="no" active="yes"/>
+<layer number="21" name="tPlace" color="7" fill="1" visible="yes" active="yes"/>
+<layer number="22" name="bPlace" color="7" fill="1" visible="yes" active="yes"/>
+<layer number="23" name="tOrigins" color="15" fill="1" visible="yes" active="yes"/>
 <layer number="24" name="bOrigins" color="15" fill="1" visible="no" active="yes"/>
-<layer number="25" name="tNames" color="7" fill="1" visible="no" active="yes"/>
-<layer number="26" name="bNames" color="7" fill="1" visible="no" active="yes"/>
-<layer number="27" name="tValues" color="7" fill="1" visible="no" active="yes"/>
-<layer number="28" name="bValues" color="7" fill="1" visible="no" active="yes"/>
+<layer number="25" name="tNames" color="7" fill="1" visible="yes" active="yes"/>
+<layer number="26" name="bNames" color="7" fill="1" visible="yes" active="yes"/>
+<layer number="27" name="tValues" color="7" fill="1" visible="yes" active="yes"/>
+<layer number="28" name="bValues" color="7" fill="1" visible="yes" active="yes"/>
 <layer number="29" name="tStop" color="7" fill="3" visible="no" active="yes"/>
 <layer number="30" name="bStop" color="7" fill="6" visible="no" active="yes"/>
@@
 <wire x1="41.33" y1="7.92" x2="34.25" y2="15" width="0.508" layer="16"/>
 </signal>
-<signal name="N$24">
+<signal name="MISO">
 <contactref element="IC6" pad="18"/>
 <contactref element="JP1" pad="2"/>
@@
 <wire x1="13.5" y1="104.5" x2="15.1" y2="104.5" width="2.54" layer="16"/>
 </signal>
-<signal name="N$66">
+<signal name="MOSI">
 <contactref element="IC6" pad="17"/>
 <contactref element="JP1" pad="1"/>
