File: boards/galvanika-board-1.0/galvanika-board-1.0.brd (EAGLE design)
At the start: 125.1 x 150 mm, 107 parts, among them IC1 LM358D, IC3 74HCT595D, IC4 74HCT595D, IC5 74HCT595D, IC6 ATMEGA48/88/168-PU, IC7 74HC595D, Q1 20MHz

Commit message: board v1
Parts:
- added R54, R55: 100k, rcl:R1206
Connections:
- net GND: now also R54.1, R55.1
- net N$12: now also R54.2
- net N$15: now also R55.2
Routing:
- net GND: track 1501.8 -> 1510.7 mm
- net N$15: track 42.6 -> 46.7 mm
- net N$12: track 68.5 -> 71.4 mm
Changed lines of the file:
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@@
 <grid distance="0.25" unitdist="mm" unit="mm" style="lines" multiple="1" display="yes" altdistance="5" altunitdist="mil" altunit="mil"/>
 <layers>
-<layer number="1" name="Top" color="4" fill="1" visible="no" active="yes"/>
+<layer number="1" name="Top" color="4" fill="1" visible="yes" active="yes"/>
 <layer number="2" name="Route2" color="16" fill="1" visible="no" active="no"/>
 <layer number="3" name="Route3" color="17" fill="1" visible="no" active="no"/>
@@
 <layer number="17" name="Pads" color="2" fill="1" visible="yes" active="yes"/>
 <layer number="18" name="Vias" color="2" fill="1" visible="yes" active="yes"/>
-<layer number="19" name="Unrouted" color="6" fill="1" visible="no" active="yes"/>
+<layer number="19" name="Unrouted" color="6" fill="1" visible="yes" active="yes"/>
 <layer number="20" name="Dimension" color="24" fill="1" visible="yes" active="yes"/>
-<layer number="21" name="tPlace" color="7" fill="1" visible="no" active="yes"/>
-<layer number="22" name="bPlace" color="7" fill="1" visible="no" active="yes"/>
-<layer number="23" name="tOrigins" color="15" fill="1" visible="no" active="yes"/>
-<layer number="24" name="bOrigins" color="15" fill="1" visible="no" active="yes"/>
-<layer number="25" name="tNames" color="7" fill="1" visible="no" active="yes"/>
-<layer number="26" name="bNames" color="7" fill="1" visible="no" active="yes"/>
+<layer number="21" name="tPlace" color="7" fill="1" visible="yes" active="yes"/>
+<layer number="22" name="bPlace" color="7" fill="1" visible="yes" active="yes"/>
+<layer number="23" name="tOrigins" color="15" fill="1" visible="yes" active="yes"/>
+<layer number="24" name="bOrigins" color="15" fill="1" visible="yes" active="yes"/>
+<layer number="25" name="tNames" color="7" fill="1" visible="yes" active="yes"/>
+<layer number="26" name="bNames" color="7" fill="1" visible="yes" active="yes"/>
 <layer number="27" name="tValues" color="7" fill="1" visible="no" active="yes"/>
 <layer number="28" name="bValues" color="7" fill="1" visible="no" active="yes"/>
@@
 <layer number="37" name="tTest" color="7" fill="1" visible="no" active="yes"/>
 <layer number="38" name="bTest" color="7" fill="1" visible="no" active="yes"/>
-<layer number="39" name="tKeepout" color="4" fill="11" visible="no" active="yes"/>
-<layer number="40" name="bKeepout" color="1" fill="11" visible="no" active="yes"/>
-<layer number="41" name="tRestrict" color="4" fill="10" visible="no" active="yes"/>
-<layer number="42" name="bRestrict" color="1" fill="10" visible="no" active="yes"/>
+<layer number="39" name="tKeepout" color="4" fill="11" visible="yes" active="yes"/>
+<layer number="40" name="bKeepout" color="1" fill="11" visible="yes" active="yes"/>
+<layer number="41" name="tRestrict" color="4" fill="10" visible="yes" active="yes"/>
+<layer number="42" name="bRestrict" color="1" fill="10" visible="yes" active="yes"/>
 <layer number="43" name="vRestrict" color="2" fill="10" visible="no" active="yes"/>
 <layer number="44" name="Drills" color="7" fill="1" visible="no" active="yes"/>
@@
 <layer number="49" name="Reference" color="7" fill="1" visible="no" active="yes"/>
 <layer number="50" name="dxf" color="7" fill="1" visible="no" active="yes"/>
-<layer number="51" name="tDocu" color="7" fill="1" visible="no" active="yes"/>
-<layer number="52" name="bDocu" color="7" fill="1" visible="no" active="yes"/>
+<layer number="51" name="tDocu" color="7" fill="1" visible="yes" active="yes"/>
+<layer number="52" name="bDocu" color="7" fill="1" visible="yes" active="yes"/>
 <layer number="53" name="tGND_GNDA" color="7" fill="1" visible="no" active="no"/>
 <layer number="54" name="bGND_GNDA" color="7" fill="1" visible="no" active="no"/>
@@
 <attribute name="VALUE" x="119.04" y="12.52" size="1.27" layer="28" rot="MR270"/>
 </element>
+<element name="R54" library="rcl" package="R1206" package3d_urn="urn:adsk.eagle:package:23540/2" value="100k" x="80.5" y="127.75" smashed="yes" rot="MR270">
+<attribute name="NAME" x="79.23" y="129.02" size="1.27" layer="26" rot="MR270"/>
+<attribute name="POPULARITY" value="41" x="80.5" y="127.75" size="1.778" layer="28" rot="MR270" display="off"/>
+<attribute name="SPICEPREFIX" value="R" x="80.5" y="127.75" size="1.778" layer="28" rot="MR270" display="off"/>
+<attribute name="VALUE" x="83.04" y="129.02" size="1.27" layer="28" rot="MR270"/>
+</element>
+<element name="R55" library="rcl" package="R1206" package3d_urn="urn:adsk.eagle:package:23540/2" value="100k" x="35.25" y="118.75" smashed="yes" rot="MR180">
+<attribute name="NAME" x="33.98" y="117.48" size="1.27" layer="26" rot="MR180"/>
+<attribute name="POPULARITY" value="41" x="35.25" y="118.75" size="1.778" layer="28" rot="MR180" display="off"/>
+<attribute name="SPICEPREFIX" value="R" x="35.25" y="118.75" size="1.778" layer="28" rot="MR180" display="off"/>
+<attribute name="VALUE" x="33.98" y="121.29" size="1.27" layer="28" rot="MR180"/>
+</element>
 </elements>
 <signals>
@@
 <wire x1="29.27" y1="120.48" x2="29.27" y2="119.25" width="1.27" layer="16"/>
 <wire x1="38.825" y1="108.075" x2="33.5" y2="113.4" width="1.27" layer="16"/>
-<wire x1="33.5" y1="117" x2="33.5" y2="113.4" width="1.27" layer="16"/>
-<wire x1="33.5" y1="117" x2="31.25" y2="119.25" width="1.27" layer="16"/>
-<wire x1="31.25" y1="119.25" x2="29.27" y2="119.25" width="1.27" layer="16"/>
+<wire x1="33.5" y1="115" x2="33.5" y2="113.4" width="1.27" layer="16"/>
+<wire x1="33.5" y1="115" x2="29.52" y2="118.98" width="1.27" layer="16"/>
+<wire x1="29.27" y1="119.25" x2="29.27" y2="118.73" width="1.27" layer="16"/>
 <wire x1="4.07" y1="7.94" x2="4.07" y2="0.705" width="1.27" layer="16"/>
 <wire x1="4.07" y1="0.705" x2="4" y2="0.635" width="1.27" layer="16"/>
@@
 <vertex x="70.75" y="140"/>
 <vertex x="70.75" y="136.5"/>
-<vertex x="80.5" y="126.75"/>
-<vertex x="90" y="126.75"/>
+<vertex x="76.5" y="130.75"/>
+<vertex x="86" y="130.75"/>
 <vertex x="83" y="133.75"/>
 <vertex x="83" y="137.75"/>
@@
 <wire x1="27" y1="53" x2="27" y2="54.85" width="1.27" layer="16"/>
 <wire x1="61.711184375" y1="121.711184375" x2="61.711184375" y2="122.905" width="0.508" layer="16"/>
+<contactref element="R54" pad="1"/>
+<contactref element="R55" pad="1"/>
+<wire x1="80.5" y1="129.172" x2="80.5" y2="131.33" width="0.508" layer="16"/>
+<wire x1="80.5" y1="131.33" x2="82.71" y2="133.54" width="0.508" layer="16"/>
+<wire x1="33.828" y1="118.75" x2="33.118" y2="118.75" width="0.508" layer="16"/>
+<wire x1="33.118" y1="118.75" x2="33.098" y2="118.73" width="0.508" layer="16"/>
+<wire x1="33.098" y1="118.73" x2="29.27" y2="118.73" width="0.508" layer="16"/>
+<wire x1="41.79" y1="149.365" x2="39.7" y2="149.365" width="0" layer="19" extent="16-16"/>
+<wire x1="112.5" y1="0.635" x2="112.385" y2="0.635" width="0" layer="19" extent="16-16"/>
 </signal>
 <signal name="N$10">
@@
 <contactref element="R8" pad="1"/>
 <contactref element="VT6" pad="G"/>
-<wire x1="84" y1="123.54" x2="80.46" y2="123.54" width="1.27" layer="16"/>
-<wire x1="80.46" y1="123.54" x2="71" y2="133" width="1.27" layer="16"/>
-<wire x1="71" y1="133" x2="50.5" y2="133" width="1.27" layer="16"/>
+<wire x1="84" y1="123.54" x2="80.25" y2="123.54" width="1.27" layer="16"/>
+<wire x1="80.25" y1="123.54" x2="78.21" y2="123.54" width="1.27" layer="16"/>
+<wire x1="78.21" y1="123.54" x2="68.75" y2="133" width="1.27" layer="16"/>
+<wire x1="68.75" y1="133" x2="50.5" y2="133" width="1.27" layer="16"/>
 <wire x1="24.75" y1="124" x2="23.83" y2="124.92" width="1.27" layer="16"/>
 <wire x1="23.83" y1="125.25" x2="23.83" y2="124.92" width="1.27" layer="16"/>
 <wire x1="42.25" y1="133" x2="45" y2="133" width="1.27" layer="16"/>
-<wire x1="24.75" y1="124" x2="30.5" y2="124" width="1.27" layer="16"/>
-<wire x1="30.5" y1="124" x2="33.25" y2="124" width="1.27" layer="16"/>
+<wire x1="24.75" y1="124" x2="33.25" y2="124" width="1.27" layer="16"/>
 <wire x1="33.25" y1="124" x2="42.25" y2="133" width="1.27" layer="16"/>
 <via x="45" y="133" extent="1-16" drill="0.8" diameter="1.6"/>
 <wire x1="45" y1="133" x2="50.5" y2="133" width="1.27" layer="1"/>
 <via x="50.5" y="133" extent="1-16" drill="0.8" diameter="1.6"/>
+<contactref element="R54" pad="2"/>
+<wire x1="80.5" y1="126.328" x2="80.5" y2="123.79" width="0.508" layer="16"/>
+<wire x1="80.5" y1="123.79" x2="80.25" y2="123.54" width="0.508" layer="16"/>
 </signal>
 <signal name="N$15">
@@
 <wire x1="36.25" y1="106.5" x2="36.25" y2="102.75" width="0.6096" layer="16"/>
 <wire x1="56.82" y1="98.75" x2="40.25" y2="98.75" width="0.508" layer="16"/>
-<wire x1="36.25" y1="114" x2="36.25" y2="115.71" width="1.27" layer="16"/>
-<wire x1="39" y1="118.46" x2="36.25" y2="115.71" width="1.27" layer="16"/>
-<wire x1="41" y1="118.46" x2="39" y2="118.46" width="1.27" layer="16"/>
+<wire x1="41" y1="118.46" x2="41" y2="117.46" width="1.27" layer="16"/>
+<wire x1="36.25" y1="114" x2="37.54" y2="114" width="1.27" layer="16"/>
+<wire x1="41" y1="117.46" x2="37.54" y2="114" width="1.27" layer="16"/>
+<contactref element="R55" pad="2"/>
+<wire x1="41" y1="118.46" x2="40.75" y2="118.71" width="0.508" layer="16"/>
+<wire x1="40.75" y1="118.71" x2="36.712" y2="118.71" width="0.508" layer="16"/>
+<wire x1="36.712" y1="118.71" x2="36.672" y2="118.75" width="0.508" layer="16"/>
 </signal>
 <signal name="N$62">
