File: boards/galvanika-board-2.0/galvanika-board-2.0.sch (EAGLE design)
At the start: 176 parts, among them IC1 LM358D, IC2 LM358D, IC3 LM358D

Commit message: board v2
Parts:
- added JP1: (no value), pinhead:PINHD-1X7
- added XS4, XS6: KLS2-2, dragberry:KLS2-2
- added XS5, XS7: CWF-2, dragberry:CWF-2
- R1: value 100K -> (none)
- R10, R37, R67: device rcl:R-EU_0207/10 -> dragberry:SQP-5W-2
- R13, R70: value 2k -> 240; device pot:3RP/1610N -> rcl:R-EU_0207/10
- R14, R71: value 2k -> (none); device pot:3RP/1610N -> rcl:R-EU_0207/10
- R15, R45, R72: value (none) -> 2k; device rcl:R-EU_R1206 -> pot:3RP/1610N
- R16, R46, R73: value 330 -> 2k; device rcl:R-EU_0207/10 -> pot:3RP/1610N
- R17, R47, R74: device dragberry:R0904N -> rcl:R-EU_R1206
- R19, R49, R76: device rcl:R-EU_R1206 -> dragberry:R0904N
- R2: value 100k -> (none)
- R20, R50, R77: value 100k -> 330
- R21, R51, R78: value 100k -> (none); device rcl:R-EU_0207/10 -> rcl:R-EU_R1206
- R22, R23, R52, R53, R79, R80: value 0.1 -> 100k; device rcl:R-EU_0411/12 -> rcl:R-EU_0207/10
- R24, R54, R81: value 100K -> 0.1; device rcl:R-EU_R1206 -> rcl:R-EU_0411/12
- R25, R55, R82: value 10K -> 0.1; device rcl:R-EU_R1206 -> rcl:R-EU_0411/12
- R26, R33, R56, R6, R63, R83: value 10K -> 100K
- R27, R57, R84: value 100K -> 10K
- R28, R58: value 100K -> 10K; device rcl:R-EU_0207/10 -> rcl:R-EU_R1206
- R29, R59: value 100k -> 100K; device rcl:R-EU_0207/10 -> rcl:R-EU_R1206
- R3, R30, R60: value 100k -> 100K
- R31, R4, R61: value 100K -> 100k
- R34, R64, R7: value 10k -> 100k
- R35, R65, R8: value (none) -> 10K; device dragberry:SQP-5W-2 -> rcl:R-EU_0207/10
- R36, R66, R9: value 240 -> 10k
- R40: value (none) -> 240; device rcl:R-EU_R1206 -> rcl:R-EU_0207/10
- R41: device rcl:R-EU_R1206 -> rcl:R-EU_0207/10
- R43, R44: value 2k -> (none); device pot:3RP/1610N -> rcl:R-EU_R1206
- R85: value (none) -> 10K; device rcl:R-EU_0207/10 -> rcl:R-EU_R1206
- R86: value (none) -> 100K; device rcl:R-EU_0207/10 -> rcl:R-EU_R1206
- XS1, XS3: value KLS2-2 -> CWF-2; device dragberry:KLS2-2 -> dragberry:CWF-2
Connections:
- removed net BRANCH-CTRL1: D8.CATHODE, R34.2, SA7.P
- removed net BRANCH-CTRL2: D13.CATHODE, R64.2, SA12.P
- new net BRANCH-CTRL-B: D8.CATHODE, DD1.PA12, R36.2, SA7.P
- new net BRANCH-CTRL-C: D13.CATHODE, DD1.PA11, R66.2, SA12.P
- new net N$17: DD1.PB12, JP1.7
- new net N$28: DD1.PB13, JP1.6
- new net N$32: DD1.PB14, JP1.5
- new net N$35: DD1.PB15, JP1.4
- new net N$45: DD1.PA8, JP1.3
- new net N$48: DD1.PA9, JP1.2
- new net N$49: DD1.PA10, JP1.1
- net +12V: now also R3.2, R30.2, R31.2, R4.2, R60.2, R61.2, XS7.1; no longer R1.2, R2.2, R28.2, R29.2, R58.2, R59.2
- net A-LEFT: now also R25.2; no longer R23.2
- net A-LEFT1: now also R55.2; no longer R53.2
- net A-LEFT2: now also R82.2; no longer R80.2
- net A-RIGHT: now also R24.2; no longer R22.2
- net A-RIGHT1: now also R54.2; no longer R52.2
- net A-RIGHT2: now also R81.2; no longer R79.2
- net ADC0: now also R19.3; no longer R17.3
- net ADC1: now also R49.3; no longer R47.3
- net ADC2: now also R26.1; no longer R24.1
- net ADC3: now also R29.2; no longer R27.2
- net ADC4: now also R76.3; no longer R74.3
- net ADC5: now also R59.2; no longer R57.2
- net ADC6: now also R56.1; no longer R54.1
- net ADC7: now also R83.1; no longer R81.1
- net ADC8: now also R86.2; no longer R84.2
- net BRANCH-CTRL-A: now also DD1.PA15, R9.2; no longer R7.2
- net GND: now also R15.A, R16.A, R2.1, R24.1, R25.1, R27.2, R28.1, R43.1, R44.1, R45.A, R46.A, R54.1, R55.1, R57.2, R58.1, R72.A, R73.A, R81.1, R82.1, R84.2, R85.1, XS7.2; no longer R13.A, R14.A, R19.1, R20.1, R25.2, R26.1, R40.1, R41.1, R43.A, R44.A, R49.1, R50.1, R55.2, R56.1, R70.A, R71.A, R76.1, R77.1, R82.2, R83.1, R86.1
- net MODE-CTRL-A: now also DD1.PB5, R17.2; no longer DD1.PB6, R15.2
- net MODE-CTRL-B: now also DD1.PB4, R47.2; no longer DD1.PB5, R45.2
- net MODE-CTRL-C: now also DD1.PB3, R74.2; no longer DD1.PB4, R72.2
- net N$1: now also R3.1; no longer R1.1
- net N$10: now also R15.S; no longer R13.S
- net N$11: now also DD1.PB6; no longer DD1.PB7
- net N$12: now also R18.1, R22.2; no longer R16.1, R20.2
- net N$13: now also R10G$1.1, R10G$2.1; no longer R8G$1.1, R8G$2.1
- net N$14: now also R10G$1.2; no longer R8G$1.2
- net N$15: now also R20.2, R23.2; no longer R18.2, R21.2
- net N$16: now also R7.1; no longer R5.1
- net N$18: now also R36.1; no longer R34.1
- net N$19: now also R14.1; no longer R12.1
- net N$2: now also DD1.PB7; no longer DD1.PB8
- net N$20: now also R4.1; no longer R2.1
- net N$21: now also R13.1, R16.E; no longer R11.1, R14.E
- net N$22: now also R39.1; no longer R37.1
- net N$23: now also R16.S; no longer R14.S
- net N$24: now also R45.S; no longer R43.S
- net N$25: now also R37G$1.1, R37G$2.1; no longer R35G$1.1, R35G$2.1
- net N$26: now also R26.2, R27.1; no longer R24.2, R25.1
- net N$27: now also R28.2, R29.1; no longer R26.2, R27.1
- net N$29: now also R46.S; no longer R44.S
- net N$3: now also R10G$2.2; no longer R8G$2.2
- net N$30: now also R41.1; no longer R39.1
- net N$31: now also R31.1; no longer R29.1
- net N$33: now also R56.2, R57.1; no longer R54.2, R55.1
- net N$34: now also R58.2, R59.1; no longer R56.2, R57.1
- net N$36: now also XS3.1, XS4.1; no longer XS2.1
- net N$37: now also R37G$2.2; no longer R35G$2.2
- net N$38: now also R37G$1.2; no longer R35G$1.2
- net N$39: now also XS3.2, XS4.2; no longer XS2.2
- net N$4: now also R1.1, R2.2; no longer R85.1, R86.2
- net N$40: now also R48.1, R52.2; no longer R46.1, R50.2
- net N$41: now also R50.2, R53.2; no longer R48.2, R51.2
- net N$42: now also R38.1, R45.E; no longer R36.1, R43.E
- net N$43: now also R40.1, R46.E; no longer R38.1, R44.E
- net N$46: now also R32.1, R33.1; no longer R30.1, R31.1
- net N$47: now also R34.1; no longer R32.1
- net N$5: now also R30.1; no longer R28.1
- net N$51: now also R60.1; no longer R58.1
- net N$53: now also R66.1; no longer R64.1
- net N$54: now also R69.1; no longer R67.1
- net N$55: now also R72.S; no longer R70.S
- net N$56: now also R67G$1.1, R67G$2.1; no longer R65G$1.1, R65G$2.1
- net N$57: now also R73.S; no longer R71.S
- net N$58: now also R71.1; no longer R69.1
- net N$59: now also R61.1; no longer R59.1
- net N$6: now also R9.1; no longer R7.1
- net N$60: now also XS2.1
- net N$63: now also XS2.2
- net N$64: now also R83.2, R84.1; no longer R81.2, R82.1
- net N$66: now also R85.2, R86.1; no longer R83.2, R84.1
- net N$68: now also XS5.1, XS6.1; no longer XS3.1
- net N$69: now also R67G$2.2; no longer R65G$2.2
- net N$7: now also R5.1, R6.1; no longer R3.1, R4.1
- net N$70: now also R67G$1.2; no longer R65G$1.2
- net N$71: now also XS5.2, XS6.2; no longer XS3.2
- net N$72: now also R75.1, R79.2; no longer R73.1, R77.2
- net N$73: now also R77.2, R80.2; no longer R75.2, R78.2
- net N$74: now also R68.1, R72.E; no longer R66.1, R70.E
- net N$75: now also R70.1, R73.E; no longer R68.1, R71.E
- net N$78: now also R62.1, R63.1; no longer R60.1, R61.1
- net N$79: now also R64.1; no longer R62.1
- net N$8: now also R12.1; no longer R10.1
- net N$84: now also R19.1, R21.2; no longer R17.1, R19.2
- net N$87: now also R49.1, R51.2; no longer R47.1, R49.2
- net N$9: now also R11.1, R15.E; no longer R13.E, R9.1
- net N$92: now also R76.1, R78.2; no longer R74.1, R76.2
- net N$95: now also DD1.PB8; no longer DD1.PB9
- net N$96: now also DD1.PB9; no longer DD1.5V
- net POWER-CTRL-A: now also R44.2; no longer R42.2
- net POWER-CTRL-B: now also R43.2; no longer R41.2
- net POWER-CTRL-C: now also R42.2; no longer R40.2
- net RIGHT-EN: now also R8.1; no longer R6.1
- net RIGHT-EN1: now also R35.1; no longer R33.1
- net RIGHT-EN2: now also R65.1; no longer R63.1
- net VCC: now also R1.2, R17.1, R19.2, R34.2, R35.2, R47.1, R49.2, R64.2, R65.2, R7.2, R74.1, R76.2, R8.2; no longer R15.1, R17.2, R3.2, R30.2, R31.2, R4.2, R45.1, R47.2, R60.2, R61.2, R72.1, R74.2, R85.2
- net VI-LEFT: now also R12.2, R20.1; no longer R10.2, R18.1
- net VI-LEFT1: now also R39.2, R50.1; no longer R37.2, R48.1
- net VI-LEFT2: now also R69.2, R77.1; no longer R67.2, R75.1
- net VI-RIGHT: now also R14.2, R18.2; no longer R12.2, R16.2
- net VI-RIGHT1: now also R41.2, R48.2; no longer R39.2, R46.2
- net VI-RIGHT2: now also R71.2, R75.2; no longer R69.2, R73.2
- net VO-LEFT: now also R11.2; no longer R9.2
- net VO-LEFT1: now also R38.2; no longer R36.2
- net VO-LEFT2: now also R68.2; no longer R66.2
- net VO-RIGHT: now also R13.2; no longer R11.2
- net VO-RIGHT1: now also R40.2; no longer R38.2
- net VO-RIGHT2: now also R70.2; no longer R68.2
Other:
- moved on the sheet: R1, R10G$1, R11, R12, R18, R2, R20, R21, R22, R23, R24, R25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

Commit message: stm32 bath 2
Parts:
- added R87, R88, R89: 510, rcl:R-EU_R1206
- C13, C5, C9: value (none) -> 1u
- R17, R47, R74: value (none) -> 4.7k
- R21, R51, R78: value (none) -> 100
- R22, R23, R31, R52, R53, R61, R79: value 100k -> 3.3k
- R3: value 100K -> 3.3K
- R30, R60: value 100K -> 3.3k
- R32, R34, R5, R62, R64, R7: value 100k -> 680k
- R33, R6, R63: value 100K -> 680K
- R4: value 100k -> 3.3K
- R42, R43, R44: value (none) -> 1k
- R80: value 100k -> 51k
- R82: value 0.1 -> 3.3k
Connections:
- net MODE-CTRL-A: now also R87.1; no longer C5.1, R17.2, SA6.1
- net MODE-CTRL-B: now also R88.1; no longer C9.1, R47.2, SA11.1
- net MODE-CTRL-C: now also R89.1; no longer C13.1, R74.2, SA16.1
- net N$17: now also C5.1, R17.2, R87.2, SA6.1; no longer DD1.PB12, JP1.7
- net N$28: now also C9.1, R47.2, R88.2, SA11.1; no longer DD1.PB13, JP1.6
- net N$32: now also C13.1, R74.2, R89.2, SA16.1; no longer DD1.PB14, JP1.5
- net PWM-CTRL-A: now also DD1.PB13; no longer DD1.PC13
- net PWM-CTRL-B: now also DD1.PB14; no longer DD1.PC14
- net PWM-CTRL-C: now also DD1.PB12; no longer DD1.PC15
Other:
- moved on the sheet: R43

Commit message: board 2.1
Parts:
- removed JP1: (no value), pinhead:PINHD-1X7
- added JP2: (no value), pinhead:PINHD-1X4
- DA3, DA5, DA7: value LM338TO220-SK29-38S -> LM338TO-220-23X16X40; device dragberry:LM338TO220-SK29-38S -> dragberry:LM338TO-220-23X16X40
- SA1: value KCD11-101-H -> KCD11-101V; device dragberry:KCD11-101-H -> dragberry:KCD11-101V
Connections:
- net +12V: now also SA1.O; no longer SA1.S
- net N$35: now also JP2.4; no longer JP1.4
- net N$45: now also JP2.3; no longer JP1.3
- net N$48: now also JP2.2; no longer JP1.2
- net N$49: now also JP2.1; no longer JP1.1
Changed lines of the file:
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@@
 <part name="VT5" library="dragberry" deviceset="2N2222" device="" package3d_urn="urn:adsk.eagle:package:28523/2"/>
 <part name="DA2" library="dragberry" deviceset="LM338" device="TO220-SK29-38S"/>
-<part name="DA3" library="dragberry" deviceset="LM338" device="TO220-SK29-38S"/>
+<part name="DA3" library="dragberry" deviceset="LM338" device="TO-220-23X16X40" value="LM338TO-220-23X16X40"/>
 <part name="XS2" library="dragberry" deviceset="KLS2-2" device=""/>
 <part name="R10" library="dragberry" deviceset="SQP-5W-2" device=""/>
@@
 <part name="R15" library="pot" library_urn="urn:adsk.eagle:library:331" deviceset="3RP/1610N" device="" package3d_urn="urn:adsk.eagle:package:22726/1" value="2k"/>
 <part name="R16" library="pot" library_urn="urn:adsk.eagle:library:331" deviceset="3RP/1610N" device="" package3d_urn="urn:adsk.eagle:package:22726/1" value="2k"/>
-<part name="SA1" library="dragberry" deviceset="KCD11-101-H" device=""/>
+<part name="SA1" library="dragberry" deviceset="KCD11-101" device="V"/>
 <part name="SA2" library="dragberry" deviceset="SS12D00" device="DIP"/>
 <part name="SA4" library="dragberry" deviceset="SS12D00" device="DIP"/>
@@
 <part name="VT9" library="dragberry" deviceset="AOD403" device=""/>
 <part name="DA4" library="dragberry" deviceset="LM338" device="TO220-SK29-38S"/>
-<part name="DA5" library="dragberry" deviceset="LM338" device="TO220-SK29-38S"/>
+<part name="DA5" library="dragberry" deviceset="LM338" device="TO-220-23X16X40" value="LM338TO-220-23X16X40"/>
 <part name="XS4" library="dragberry" deviceset="KLS2-2" device=""/>
 <part name="R37" library="dragberry" deviceset="SQP-5W-2" device=""/>
@@
 <part name="VT16" library="dragberry" deviceset="AOD403" device=""/>
 <part name="DA6" library="dragberry" deviceset="LM338" device="TO220-SK29-38S"/>
-<part name="DA7" library="dragberry" deviceset="LM338" device="TO220-SK29-38S"/>
+<part name="DA7" library="dragberry" deviceset="LM338" device="TO-220-23X16X40" value="LM338TO-220-23X16X40"/>
 <part name="XS6" library="dragberry" deviceset="KLS2-2" device=""/>
 <part name="R67" library="dragberry" deviceset="SQP-5W-2" device=""/>
@@
 <part name="XS5" library="dragberry" deviceset="CWF-2" device=""/>
 <part name="XS7" library="dragberry" deviceset="CWF-2" device=""/>
-<part name="JP1" library="pinhead" library_urn="urn:adsk.eagle:library:325" deviceset="PINHD-1X7" device="" package3d_urn="urn:adsk.eagle:package:22477/2"/>
 <part name="R87" library="rcl" deviceset="R-EU_" device="R1206" package3d_urn="urn:adsk.eagle:package:23540/2" value="510"/>
 <part name="R88" library="rcl" deviceset="R-EU_" device="R1206" package3d_urn="urn:adsk.eagle:package:23540/2" value="510"/>
 <part name="R89" library="rcl" deviceset="R-EU_" device="R1206" package3d_urn="urn:adsk.eagle:package:23540/2" value="510"/>
+<part name="JP2" library="pinhead" library_urn="urn:adsk.eagle:library:325" deviceset="PINHD-1X4" device="" package3d_urn="urn:adsk.eagle:package:22407/2"/>
 </parts>
 <sheets>
@@
 <attribute name="VALUE" x="62.23" y="144.78" size="1.778" layer="96"/>
 </instance>
-<instance part="JP1" gate="A" x="-231.14" y="-124.46" smashed="yes" rot="R180">
-<attribute name="NAME" x="-224.79" y="-135.255" size="1.778" layer="95" rot="R180"/>
-<attribute name="VALUE" x="-224.79" y="-111.76" size="1.778" layer="96" rot="R180"/>
-</instance>
 <instance part="R87" gate="G$1" x="-40.64" y="-2.54" smashed="yes">
 <attribute name="NAME" x="-44.45" y="-1.0414" size="1.778" layer="95"/>
@@
 <attribute name="NAME" x="-44.45" y="-349.0214" size="1.778" layer="95"/>
 <attribute name="VALUE" x="-44.45" y="-353.822" size="1.778" layer="96"/>
+</instance>
+<instance part="JP2" gate="A" x="-238.76" y="-127" smashed="yes" rot="R180">
+<attribute name="NAME" x="-232.41" y="-135.255" size="1.778" layer="95" rot="R180"/>
+<attribute name="VALUE" x="-232.41" y="-119.38" size="1.778" layer="96" rot="R180"/>
 </instance>
 </instances>
@@
 <junction x="76.2" y="152.4"/>
 <wire x1="76.2" y1="152.4" x2="76.2" y2="157.48" width="0.1524" layer="91"/>
-<pinref part="SA1" gate="G$1" pin="S"/>
-<wire x1="55.88" y1="149.86" x2="55.88" y2="152.4" width="0.1524" layer="91"/>
 <wire x1="55.88" y1="152.4" x2="66.04" y2="152.4" width="0.1524" layer="91"/>
 <pinref part="DA1" gate="G$1" pin="VI"/>
@@
 <wire x1="66.04" y1="152.4" x2="76.2" y2="152.4" width="0.1524" layer="91"/>
 <junction x="66.04" y="152.4"/>
+<pinref part="SA1" gate="G$1" pin="O"/>
+<wire x1="55.88" y1="154.94" x2="55.88" y2="152.4" width="0.1524" layer="91"/>
 </segment>
 <segment>
@@
 <segment>
 <pinref part="DD1" gate="G$1" pin="PB15"/>
-<pinref part="JP1" gate="A" pin="4"/>
-<wire x1="-218.44" y1="-124.46" x2="-228.6" y2="-124.46" width="0.1524" layer="91"/>
+<wire x1="-218.44" y1="-124.46" x2="-236.22" y2="-124.46" width="0.1524" layer="91"/>
+<pinref part="JP2" gate="A" pin="4"/>
 </segment>
 </net>
@@
 <segment>
 <pinref part="DD1" gate="G$1" pin="PA8"/>
-<pinref part="JP1" gate="A" pin="3"/>
-<wire x1="-218.44" y1="-127" x2="-228.6" y2="-127" width="0.1524" layer="91"/>
+<wire x1="-218.44" y1="-127" x2="-236.22" y2="-127" width="0.1524" layer="91"/>
+<pinref part="JP2" gate="A" pin="3"/>
 </segment>
 </net>
@@
 <segment>
 <pinref part="DD1" gate="G$1" pin="PA9"/>
-<pinref part="JP1" gate="A" pin="2"/>
-<wire x1="-218.44" y1="-129.54" x2="-228.6" y2="-129.54" width="0.1524" layer="91"/>
+<wire x1="-218.44" y1="-129.54" x2="-236.22" y2="-129.54" width="0.1524" layer="91"/>
+<pinref part="JP2" gate="A" pin="2"/>
 </segment>
 </net>
 <net name="N$49" class="0">
 <segment>
-<pinref part="JP1" gate="A" pin="1"/>
 <pinref part="DD1" gate="G$1" pin="PA10"/>
-<wire x1="-228.6" y1="-132.08" x2="-218.44" y2="-132.08" width="0.1524" layer="91"/>
-</segment>
-</net>
+<wire x1="-236.22" y1="-132.08" x2="-218.44" y2="-132.08" width="0.1524" layer="91"/>
+<pinref part="JP2" gate="A" pin="1"/>
+</segment>
+</net>
