File: boards/galvanika-board-2.0/galvanika-board-2.0.brd (EAGLE design)
At the start: 250 x 150 mm, 176 parts, among them IC1 LM358D, IC2 LM358D, IC3 LM358D

Commit message: board v2
Parts:
- added JP1: (no value), pinhead:1X07
- added XS4, XS6: KLS2-2, dragberry:KLS2-2
- added XS5, XS7: CWF-2, dragberry:CWF-2
- R1: value 100K -> (none)
- R10, R37, R67: device rcl:0207/10 -> dragberry:SQP-5W-2
- R13, R70: value 2k -> 240; device pot:3RP/1610N -> rcl:0207/10
- R14, R71: value 2k -> (none); device pot:3RP/1610N -> rcl:0207/10
- R15, R45, R72: value (none) -> 2k; device rcl:R1206 -> pot:3RP/1610N
- R16, R46, R73: value 330 -> 2k; device rcl:0207/10 -> pot:3RP/1610N
- R17, R47, R74: device dragberry:R0904N -> rcl:R1206
- R19, R49, R76: device rcl:R1206 -> dragberry:R0904N
- R2: value 100k -> (none)
- R20, R50, R77: value 100k -> 330
- R21, R51, R78: value 100k -> (none); device rcl:0207/10 -> rcl:R1206
- R22, R23, R52, R53, R79, R80: value 0.1 -> 100k; device rcl:0411/12 -> rcl:0207/10
- R24, R54, R81: value 100K -> 0.1; device rcl:R1206 -> rcl:0411/12
- R25, R55, R82: value 10K -> 0.1; device rcl:R1206 -> rcl:0411/12
- R26, R33, R56, R6, R63, R83: value 10K -> 100K
- R27, R57, R84: value 100K -> 10K
- R28, R58: value 100K -> 10K; device rcl:0207/10 -> rcl:R1206
- R29, R59: value 100k -> 100K; device rcl:0207/10 -> rcl:R1206
- R3, R30, R60: value 100k -> 100K
- R31, R4, R61: value 100K -> 100k
- R34, R64, R7: value 10k -> 100k
- R35, R65, R8: value (none) -> 10K; device dragberry:SQP-5W-2 -> rcl:0207/10
- R36, R66, R9: value 240 -> 10k
- R40: value (none) -> 240; device rcl:R1206 -> rcl:0207/10
- R41: device rcl:R1206 -> rcl:0207/10
- R43, R44: value 2k -> (none); device pot:3RP/1610N -> rcl:R1206
- R85: value (none) -> 10K; device rcl:0207/10 -> rcl:R1206
- R86: value (none) -> 100K; device rcl:0207/10 -> rcl:R1206
- XS1, XS3: value KLS2-2 -> CWF-2; device dragberry:KLS2-2 -> dragberry:CWF-2
- moved R46 166.4 mm to (6.00, 55.0)
- moved R73 162.9 mm to (5.75, 100.0), turned to 270 degrees
- moved R16 162.3 mm to (5.75, 10.0)
- moved R78 160.0 mm to (23.5, 97.5), flipped to the bottom, turned to 180 degrees
- moved R71 159.7 mm to (163.1, 127.4), turned to 180 degrees
- moved R21 157.7 mm to (22.5, 17.5), flipped to the bottom, turned to 180 degrees
- moved R14 157.5 mm to (163.0, 18.5), turned to 180 degrees
- moved R51 155.2 mm to (22.8, 62.8), flipped to the bottom, turned to 180 degrees
- moved R86 153.4 mm to (217.5, 122.5), flipped to the bottom
- moved R85 143.0 mm to (207.5, 129.2), flipped to the bottom, turned to 270 degrees
- moved R2 129.8 mm to (64.5, 133.8)
- moved R13 127.9 mm to (132.2, 9.75), turned to 90 degrees
- moved R70 127.1 mm to (132.8, 114.8), turned to 90 degrees
- moved R1 123.9 mm to (64.5, 130.5), turned to 180 degrees
- moved R8 116.9 mm to (101.2, 32.5), flipped to the bottom
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Connections:
- removed net BRANCH-CTRL1: D8.C, R34.2, SA7.1$P
- removed net BRANCH-CTRL2: D13.C, R64.2, SA12.1$P
- new net BRANCH-CTRL-B: D8.C, DD1.P$9, R36.2, SA7.1$P
- new net BRANCH-CTRL-C: D13.C, DD1.P$8, R66.2, SA12.1$P
- new net N$17: DD1.P$1, JP1.7
- new net N$28: DD1.P$2, JP1.6
- new net N$32: DD1.P$3, JP1.5
- new net N$35: DD1.P$4, JP1.4
- new net N$45: DD1.P$5, JP1.3
- new net N$48: DD1.P$6, JP1.2
- new net N$49: DD1.P$7, JP1.1
- net +12V: now also R3.2, R30.2, R31.2, R4.2, R60.2, R61.2, XS7.P$1; no longer R1.2, R2.2, R28.2, R29.2, R58.2, R59.2
- net A-LEFT: now also R25.2; no longer R23.2
- net A-LEFT1: now also R55.2; no longer R53.2
- net A-LEFT2: now also R82.2; no longer R80.2
- net A-RIGHT: now also R24.2; no longer R22.2
- net A-RIGHT1: now also R54.2; no longer R52.2
- net A-RIGHT2: now also R81.2; no longer R79.2
- net ADC0: now also R19.2; no longer R17.2
- net ADC1: now also R49.2; no longer R47.2
- net ADC2: now also R26.1; no longer R24.1
- net ADC3: now also R29.2; no longer R27.2
- net ADC4: now also R76.2; no longer R74.2
- net ADC5: now also R59.2; no longer R57.2
- net ADC6: now also R56.1; no longer R54.1
- net ADC7: now also R83.1; no longer R81.1
- net ADC8: now also R86.2; no longer R84.2
- net BRANCH-CTRL-A: now also DD1.P$10, R9.2; no longer R7.2
- net GND: now also R15.1, R16.1, R2.1, R24.1, R25.1, R27.2, R28.1, R45.1, R46.1, R54.1, R55.1, R57.2, R58.1, R72.1, R73.1, R81.1, R82.1, R84.2, R85.1, XS7.P$2; no longer R13.1, R14.1, R19.1, R20.1, R25.2, R26.1, R40.1, R41.1, R49.1, R50.1, R55.2, R56.1, R70.1, R71.1, R76.1, R77.1, R82.2, R83.1, R86.1
- net MODE-CTRL-A: now also DD1.P$13, R17.2; no longer DD1.P$14, R15.2
- net MODE-CTRL-B: now also DD1.P$12, R47.2; no longer DD1.P$13, R45.2
- net MODE-CTRL-C: now also DD1.P$11, R74.2; no longer DD1.P$12, R72.2
- net N$1: now also R3.1; no longer R1.1
- net N$10: now also R15.2; no longer R13.2
- net N$11: now also DD1.P$14; no longer DD1.P$15
- net N$12: now also R18.1, R22.2; no longer R16.1, R20.2
- net N$13: now also R10.1, R10.3; no longer R8.1, R8.3
- net N$14: now also R10.2; no longer R8.2
- net N$15: now also R20.2, R23.2; no longer R18.2, R21.2
- net N$16: now also R7.1; no longer R5.1
- net N$18: now also R36.1; no longer R34.1
- net N$19: now also R14.1; no longer R12.1
- net N$2: now also DD1.P$15; no longer DD1.P$16
- net N$20: now also R4.1; no longer R2.1
- net N$21: now also R13.1, R16.3; no longer R11.1, R14.3
- net N$22: now also R39.1; no longer R37.1
- net N$23: now also R16.2; no longer R14.2
- net N$24: now also R45.2; no longer R43.2
- net N$25: now also R37.1, R37.3; no longer R35.1, R35.3
- net N$26: now also R26.2, R27.1; no longer R24.2, R25.1
- net N$27: now also R28.2, R29.1; no longer R26.2, R27.1
- net N$29: now also R46.2; no longer R44.2
- net N$3: now also R10.4; no longer R8.4
- net N$30: now also R41.1; no longer R39.1
- net N$31: now also R31.1; no longer R29.1
- net N$33: now also R56.2, R57.1; no longer R54.2, R55.1
- net N$34: now also R58.2, R59.1; no longer R56.2, R57.1
- net N$36: now also XS3.P$1, XS4.1; no longer XS2.1
- net N$37: now also R37.4; no longer R35.4
- net N$38: now also R37.2; no longer R35.2
- net N$39: now also XS3.P$2, XS4.2; no longer XS2.2
- net N$4: now also R1.1, R2.2; no longer R85.1, R86.2
- net N$40: now also R48.1, R52.2; no longer R46.1, R50.2
- net N$41: now also R50.2, R53.2; no longer R48.2, R51.2
- net N$42: now also R38.1, R45.3; no longer R36.1, R43.3
- net N$43: now also R40.1, R46.3; no longer R38.1, R44.3
- net N$46: now also R32.1, R33.1; no longer R30.1, R31.1
- net N$47: now also R34.1; no longer R32.1
- net N$5: now also R30.1; no longer R28.1
- net N$51: now also R60.1; no longer R58.1
- net N$53: now also R66.1; no longer R64.1
- net N$54: now also R69.1; no longer R67.1
- net N$55: now also R72.2; no longer R70.2
- net N$56: now also R67.1, R67.3; no longer R65.1, R65.3
- net N$57: now also R73.2; no longer R71.2
- net N$58: now also R71.1; no longer R69.1
- net N$59: now also R61.1; no longer R59.1
- net N$6: now also R9.1; no longer R7.1
- net N$60: now also XS1.P$1, XS2.1; no longer XS1.1
- net N$63: now also XS1.P$2, XS2.2; no longer XS1.2
- net N$64: now also R83.2, R84.1; no longer R81.2, R82.1
- net N$66: now also R85.2, R86.1; no longer R83.2, R84.1
- net N$68: now also XS5.P$1, XS6.1; no longer XS3.1
- net N$69: now also R67.4; no longer R65.4
- net N$7: now also R5.1, R6.1; no longer R3.1, R4.1
- net N$70: now also R67.2; no longer R65.2
- net N$71: now also XS5.P$2, XS6.2; no longer XS3.2
- net N$72: now also R75.1, R79.2; no longer R73.1, R77.2
- net N$73: now also R77.2, R80.2; no longer R75.2, R78.2
- net N$74: now also R68.1, R72.3; no longer R66.1, R70.3
- net N$75: now also R70.1, R73.3; no longer R68.1, R71.3
- net N$78: now also R62.1, R63.1; no longer R60.1, R61.1
- net N$79: now also R64.1; no longer R62.1
- net N$8: now also R12.1; no longer R10.1
- net N$84: now also R19.1, R21.2; no longer R17.1, R19.2
- net N$87: now also R49.1, R51.2; no longer R47.1, R49.2
- net N$9: now also R11.1, R15.3; no longer R13.3, R9.1
- net N$92: now also R76.1, R78.2; no longer R74.1, R76.2
- net N$95: now also DD1.P$16; no longer DD1.P$17
- net N$96: now also DD1.P$17; no longer DD1.P$18
- net POWER-CTRL-A: now also R44.2; no longer R42.2
- net POWER-CTRL-B: now also R43.2; no longer R41.2
- net POWER-CTRL-C: now also R42.2; no longer R40.2
- net RIGHT-EN: now also R8.1; no longer R6.1
- net RIGHT-EN1: now also R35.1; no longer R33.1
- net RIGHT-EN2: now also R65.1; no longer R63.1
- net VCC: now also R1.2, R17.1, R19.3, R34.2, R35.2, R47.1, R49.3, R64.2, R65.2, R7.2, R74.1, R76.3, R8.2; no longer R15.1, R17.3, R3.2, R30.2, R31.2, R4.2, R45.1, R47.3, R60.2, R61.2, R72.1, R74.3, R85.2
- net VI-LEFT: now also R12.2, R20.1; no longer R10.2, R18.1
- net VI-LEFT1: now also R39.2, R50.1; no longer R37.2, R48.1
- net VI-LEFT2: now also R69.2, R77.1; no longer R67.2, R75.1
- net VI-RIGHT: now also R14.2, R18.2; no longer R12.2, R16.2
- net VI-RIGHT1: now also R41.2, R48.2; no longer R39.2, R46.2
- net VI-RIGHT2: now also R71.2, R75.2; no longer R69.2, R73.2
- net VO-LEFT: now also R11.2; no longer R9.2
- net VO-LEFT1: now also R38.2; no longer R36.2
- net VO-LEFT2: now also R68.2; no longer R66.2
- net VO-RIGHT: now also R13.2; no longer R11.2
- net VO-RIGHT1: now also R40.2; no longer R38.2
- net VO-RIGHT2: now also R70.2; no longer R68.2
Routing:
- net BRANCH-CTRL-B: track 0.00 -> 153.6 mm, vias 0 -> 4
- net BRANCH-CTRL-A: track 24.6 -> 118.8 mm, vias 0 -> 4
- net BRANCH-CTRL-C: track 0.00 -> 91.8 mm, vias 0 -> 2
- net BRANCH-CTRL1: track 26.7 -> 0.00 mm
- net BRANCH-CTRL2: track 18.5 -> 0.00 mm
- net GND: track 2416.3 -> 2434.6 mm
- net N$49: track 0.00 -> 9.93 mm
- net N$48: track 0.00 -> 9.93 mm
- net N$45: track 0.00 -> 9.93 mm
- net N$35: track 0.00 -> 9.93 mm
- net N$28: track 0.00 -> 9.93 mm
- net N$32: track 0.00 -> 9.93 mm
- net N$17: track 0.00 -> 9.93 mm
- net N$75: track 153.0 -> 145.7 mm
- net N$68: track 81.2 -> 88.1 mm
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Other:
- board text added: "DRAGBERRY 2021.01"
- board text added: "GALVANIKA CUPRUMBERRY V2.0"

Commit message: stm32 bath 2
Parts:
- added R87, R88, R89: 510, rcl:R1206
- C13, C5, C9: value (none) -> 1u
- R17, R47, R74: value (none) -> 4.7k
- R21, R51, R78: value (none) -> 100
- R22, R23, R31, R52, R53, R61, R79: value 100k -> 3.3k
- R3: value 100K -> 3.3K
- R30, R60: value 100K -> 3.3k
- R32, R34, R5, R62, R64, R7: value 100k -> 680k
- R33, R6, R63: value 100K -> 680K
- R4: value 100k -> 3.3K
- R42, R43, R44: value (none) -> 1k
- R80: value 100k -> 51k
- R82: value 0.1 -> 3.3k
Connections:
- net MODE-CTRL-A: now also R87.1; no longer C5.1, R17.2, SA6.P$1, SA6.P$2
- net MODE-CTRL-B: now also R88.1; no longer C9.1, R47.2, SA11.P$1, SA11.P$2
- net MODE-CTRL-C: now also R89.1; no longer C13.1, R74.2, SA16.P$1, SA16.P$2
- net N$17: now also C5.1, R17.2, R87.2, SA6.P$1, SA6.P$2; no longer DD1.P$1, JP1.7
- net N$28: now also C9.1, R47.2, R88.2, SA11.P$1, SA11.P$2; no longer DD1.P$2, JP1.6
- net N$32: now also C13.1, R74.2, R89.2, SA16.P$1, SA16.P$2; no longer DD1.P$3, JP1.5
- net PWM-CTRL-A: now also DD1.P$2; no longer DD1.P$39
- net PWM-CTRL-B: now also DD1.P$3; no longer DD1.P$38
- net PWM-CTRL-C: now also DD1.P$1; no longer DD1.P$37
Routing:
- net MODE-CTRL-C: track 124.2 -> 11.7 mm
- net N$32: track 9.93 -> 110.2 mm
- net PWM-CTRL-B: track 55.4 -> 124.8 mm, vias 4 -> 6
- net PWM-CTRL-A: track 61.0 -> 112.4 mm, vias 2 -> 4
- net PWM-CTRL-C: track 102.4 -> 67.6 mm, vias 4 -> 2
- net MODE-CTRL-B: track 44.9 -> 10.7 mm
- net N$28: track 9.93 -> 35.1 mm
- net MODE-CTRL-A: track 72.4 -> 51.5 mm
- net N$17: track 9.93 -> 19.2 mm
- net VI-LEFT2: track 66.2 -> 72.4 mm
- net N$40: track 47.0 -> 42.4 mm
- net BRANCH-CTRL-C: track 91.8 -> 89.2 mm
- net ADC0: track 89.5 -> 91.8 mm
- net ADC1: track 57.1 -> 59.4 mm
- net N$73: track 48.1 -> 49.8 mm
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Other:
- board text added: "GALVANIKA CUPRUMBERRY V2.1"
- board text removed: "GALVANIKA CUPRUMBERRY V2.0"

Commit message: board 2.1
Parts:
- removed JP1: (no value), pinhead:1X07
- added JP2: (no value), pinhead:1X04
- DA3, DA5, DA7: value LM338TO220-SK29-38S -> LM338TO-220-23X16X40; device dragberry:TO220-SK29-38S -> dragberry:TO220-23X16X40
- SA1: value KCD11-101-H -> KCD11-101V; device dragberry:KCD11-101-H -> dragberry:KCD11-101-V
- moved D5 30.5 mm to (187.5, 7.00)
- moved R82 29.5 mm to (196.8, 112.0), turned to 90 degrees
- moved R22 26.2 mm to (179.2, 35.2), turned to 270 degrees
- moved R81 22.0 mm to (196.8, 139.2), turned to 270 degrees
- moved C3 17.2 mm to (169.0, 30.5), turned to 270 degrees
- moved C7 16.9 mm to (168.2, 85.8), turned to 270 degrees
- moved C11 15.7 mm to (167.2, 139.2), turned to 270 degrees
- moved C12 15.4 mm to (164.0, 115.5), turned to 90 degrees
- moved R26 14.7 mm to (209.0, 20.5)
- moved C8 14.4 mm to (164.5, 62.2), turned to 90 degrees
- moved C4 13.4 mm to (165.8, 11.8), turned to 90 degrees
- moved R28 7.77 mm to (226.0, 20.5)
- moved R27 6.27 mm to (217.5, 13.8), turned to 180 degrees
- moved R20 5.59 mm to (173.1, 35.1)
- moved R71 5.53 mm to (168.3, 125.7)
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Connections:
- net +12V: now also SA1.1; no longer SA1.3
- net N$35: now also JP2.4; no longer JP1.4
- net N$45: now also JP2.3; no longer JP1.3
- net N$48: now also JP2.2; no longer JP1.2
- net N$49: now also JP2.1; no longer JP1.1
- net N$65: now also SA1.3; no longer SA1.2
Routing:
- net VCC: track 923.0 -> 823.0 mm, vias 12 -> 14
- net VO-RIGHT: track 91.7 -> 61.8 mm
- net N$26: track 38.4 -> 14.2 mm, vias 2 -> 0
- net N$72: track 66.4 -> 45.0 mm, vias 0 -> 2
- net A-RIGHT2: track 91.2 -> 71.4 mm
- net ADC3: track 230.8 -> 213.5 mm
- net A-LEFT2: track 63.4 -> 47.5 mm
- net VO-RIGHT1: track 70.6 -> 58.0 mm
- net ADC8: track 185.1 -> 172.7 mm
- net ADC7: track 203.3 -> 191.6 mm
- net A-RIGHT: track 41.4 -> 53.1 mm
- net VI-RIGHT1: track 160.4 -> 150.0 mm
- net A-LEFT: track 38.8 -> 48.7 mm
- net N$65: track 18.2 -> 8.43 mm
- net VO-RIGHT2: track 74.9 -> 65.4 mm
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
Commit message: stm32 board v2.1
Routing:
- net VCC: track 823.0 -> 832.8 mm
- net ADC4: track 64.5 -> 71.1 mm
- net N$57: track 158.2 -> 161.8 mm
- net N$75: track 145.7 -> 149.2 mm
- net ADC6: track 176.0 -> 173.0 mm
- net GND: track 2438.2 -> 2435.4 mm
- net N$10: track 232.6 -> 235.3 mm
- net ADC8: track 172.7 -> 174.4 mm
- net N$23: track 150.5 -> 149.0 mm
- net ADC0: track 91.8 -> 93.2 mm
- net ADC2: track 208.6 -> 207.4 mm
- net ADC7: track 191.6 -> 192.6 mm
- net N$24: track 197.5 -> 196.8 mm
- net MODE-CTRL-A: track 51.5 -> 50.8 mm
