File: boards/pump-board-1.0/pump-board-1.0.brd (EAGLE design)
At the start: 100 x 50 mm, 59 parts, among them IC1 74HC595D, IC2 74HC595D, IC3 ATMEGA48/88/168-PU, IC4 7805TV

Commit message: pump board
Parts:
- moved R19 5.45 mm to (35.1, 32.4), turned to 0 degrees
- moved VT5 2.38 mm to (36.7, 27.8)
- moved R17 1.12 mm to (42.6, 16.9)
Routing:
- net N$39: track 17.4 -> 12.7 mm
- net VCC: track 275.8 -> 272.0 mm
- net GND: track 508.9 -> 506.5 mm
- net +12V: track 27.3 -> 29.2 mm
- net N$40: track 9.46 -> 11.0 mm
- net N$52: track 108.0 -> 109.1 mm
- net N$35: track 31.4 -> 30.5 mm
- net N$31: track 129.1 -> 129.9 mm
- net N$21: track 17.8 -> 17.1 mm
- net N$33: track 136.9 -> 137.4 mm
Other:
- board text added: "2021.02"
- board text added: "CUPRUMBERRY"
- board text added: "DRAGBERRY"

Commit message: pump code
Parts:
- R18: value (none) -> 510
- R19: value (none) -> 2k
Changed lines of the file:
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@@
 <layer number="25" name="tNames" color="7" fill="1" visible="yes" active="yes"/>
 <layer number="26" name="bNames" color="7" fill="1" visible="yes" active="yes"/>
-<layer number="27" name="tValues" color="7" fill="1" visible="no" active="yes"/>
-<layer number="28" name="bValues" color="7" fill="1" visible="no" active="yes"/>
+<layer number="27" name="tValues" color="7" fill="1" visible="yes" active="yes"/>
+<layer number="28" name="bValues" color="7" fill="1" visible="yes" active="yes"/>
 <layer number="29" name="tStop" color="7" fill="3" visible="no" active="yes"/>
 <layer number="30" name="bStop" color="7" fill="6" visible="no" active="yes"/>
@@
 </element>
 <element name="R13" library="rcl" library_urn="urn:adsk.eagle:library:334" package="R1206" package3d_urn="urn:adsk.eagle:package:23540/2" value="390" x="75.94" y="11.15" smashed="yes" rot="MR0">
-<attribute name="NAME" x="77.21" y="12.42" size="1.27" layer="26" rot="MR0"/>
+<attribute name="NAME" x="77.21" y="12.52" size="1.27" layer="26" rot="MR0"/>
 <attribute name="POPULARITY" value="41" x="60.7" y="-33.3" size="1.778" layer="28" rot="MR0" display="off"/>
 <attribute name="SPICEPREFIX" value="R" x="60.7" y="-33.3" size="1.778" layer="28" rot="MR0" display="off"/>
-<attribute name="VALUE" x="77.21" y="8.61" size="1.27" layer="28" rot="MR0"/>
+<attribute name="VALUE" x="73.51" y="11.71" size="1.27" layer="28" rot="MR0"/>
 </element>
 <element name="R14" library="rcl" library_urn="urn:adsk.eagle:library:334" package="R1206" package3d_urn="urn:adsk.eagle:package:23540/2" value="390" x="75.94" y="14.4" smashed="yes" rot="MR0">
-<attribute name="NAME" x="77.21" y="15.67" size="1.27" layer="26" rot="MR0"/>
+<attribute name="NAME" x="77.11" y="15.97" size="1.27" layer="26" rot="MR0"/>
 <attribute name="POPULARITY" value="41" x="55.62" y="-30.05" size="1.778" layer="28" rot="MR0" display="off"/>
 <attribute name="SPICEPREFIX" value="R" x="55.62" y="-30.05" size="1.778" layer="28" rot="MR0" display="off"/>
-<attribute name="VALUE" x="77.21" y="11.86" size="1.27" layer="28" rot="MR0"/>
+<attribute name="VALUE" x="73.41" y="14.86" size="1.27" layer="28" rot="MR0"/>
 </element>
 <element name="R15" library="rcl" library_urn="urn:adsk.eagle:library:334" package="R1206" package3d_urn="urn:adsk.eagle:package:23540/2" value="390" x="75.94" y="17.65" smashed="yes" rot="MR0">
@@
 <attribute name="POPULARITY" value="41" x="50.54" y="-26.8" size="1.778" layer="28" rot="MR0" display="off"/>
 <attribute name="SPICEPREFIX" value="R" x="50.54" y="-26.8" size="1.778" layer="28" rot="MR0" display="off"/>
-<attribute name="VALUE" x="77.21" y="15.11" size="1.27" layer="28" rot="MR0"/>
+<attribute name="VALUE" x="73.61" y="18.21" size="1.27" layer="28" rot="MR0"/>
 </element>
 <element name="R16" library="rcl" library_urn="urn:adsk.eagle:library:334" package="R1206" package3d_urn="urn:adsk.eagle:package:23540/2" value="390" x="75.94" y="20.9" smashed="yes" rot="MR0">
@@
 <attribute name="POPULARITY" value="41" x="45.46" y="-23.55" size="1.778" layer="28" rot="MR0" display="off"/>
 <attribute name="SPICEPREFIX" value="R" x="45.46" y="-23.55" size="1.778" layer="28" rot="MR0" display="off"/>
-<attribute name="VALUE" x="77.21" y="18.36" size="1.27" layer="28" rot="MR0"/>
+<attribute name="VALUE" x="73.61" y="21.46" size="1.27" layer="28" rot="MR0"/>
 </element>
 <element name="R17" library="rcl" library_urn="urn:adsk.eagle:library:334" package="0207/10" package3d_urn="urn:adsk.eagle:package:23491/2" value="10k" x="42.59" y="16.92" smashed="yes" rot="R90">
@@
 <attribute name="VALUE" x="43.063" y="33.54" size="1.778" layer="27" ratio="10"/>
 </element>
-<element name="R18" library="rcl" library_urn="urn:adsk.eagle:library:334" package="0207/10" package3d_urn="urn:adsk.eagle:package:23491/2" value="" x="23.9" y="35.4" smashed="yes">
+<element name="R18" library="rcl" library_urn="urn:adsk.eagle:library:334" package="0207/10" package3d_urn="urn:adsk.eagle:package:23491/2" value="510" x="23.9" y="35.4" smashed="yes">
 <attribute name="NAME" x="20.852" y="36.924" size="1.27" layer="25" ratio="10"/>
 <attribute name="POPULARITY" value="81" x="23.9" y="35.4" size="1.778" layer="27" display="off"/>
@@
 <attribute name="VALUE" x="21.6394" y="34.765" size="1.27" layer="27" ratio="10"/>
 </element>
-<element name="R19" library="rcl" library_urn="urn:adsk.eagle:library:334" package="R1206" package3d_urn="urn:adsk.eagle:package:23540/2" value="" x="35.1" y="32.4" smashed="yes" rot="MR0">
+<element name="R19" library="rcl" library_urn="urn:adsk.eagle:library:334" package="R1206" package3d_urn="urn:adsk.eagle:package:23540/2" value="2k" x="35.1" y="32.4" smashed="yes" rot="MR0">
 <attribute name="NAME" x="38.148" y="33.924" size="1.27" layer="26" ratio="10" rot="MR0"/>
 <attribute name="POPULARITY" value="41" x="35.1" y="32.4" size="1.778" layer="28" rot="MR0" display="off"/>

Commit message: pump
Parts:
- added R26: (no value), rcl:R1206
- moved R19 1.50 mm to (36.6, 32.5)
- moved VT5 0.90 mm to (37.6, 27.8)
Connections:
- net N$40: now also R26.1
- net VCC: now also R26.2
Routing:
- net VCC: track 272.0 -> 275.0 mm
- net N$40: track 11.0 -> 13.7 mm
- net N$39: track 12.7 -> 11.0 mm
- net GND: track 506.5 -> 505.6 mm
Changed lines of the file:
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@@
 <attribute name="VALUE" x="10.963" y="33.38" size="1.27" layer="27" ratio="10" rot="R270"/>
 </element>
-<element name="VT5" library="dragberry" package="TO92" package3d_urn="urn:adsk.eagle:package:28523/2" value="2N2222" x="36.7" y="27.8" smashed="yes">
-<attribute name="NAME" x="39.875" y="28.435" size="1.27" layer="25" ratio="10"/>
-<attribute name="VALUE" x="39.875" y="26.53" size="1.27" layer="27" ratio="10"/>
+<element name="VT5" library="dragberry" package="TO92" package3d_urn="urn:adsk.eagle:package:28523/2" value="2N2222" x="37.6" y="27.8" smashed="yes">
+<attribute name="NAME" x="40.775" y="28.435" size="1.27" layer="25" ratio="10"/>
+<attribute name="VALUE" x="40.775" y="26.53" size="1.27" layer="27" ratio="10"/>
 </element>
 <element name="VT6" library="dragberry" package="TO220-V" package3d_urn="urn:adsk.eagle:package:29490/1" value="IRF1404" x="47" y="31" smashed="yes">
@@
 <attribute name="VALUE" x="21.6394" y="34.765" size="1.27" layer="27" ratio="10"/>
 </element>
-<element name="R19" library="rcl" library_urn="urn:adsk.eagle:library:334" package="R1206" package3d_urn="urn:adsk.eagle:package:23540/2" value="2k" x="35.1" y="32.4" smashed="yes" rot="MR0">
-<attribute name="NAME" x="38.148" y="33.924" size="1.27" layer="26" ratio="10" rot="MR0"/>
-<attribute name="POPULARITY" value="41" x="35.1" y="32.4" size="1.778" layer="28" rot="MR0" display="off"/>
-<attribute name="SPICEPREFIX" value="R" x="35.1" y="32.4" size="1.778" layer="28" rot="MR0" display="off"/>
-<attribute name="VALUE" x="37.3606" y="31.765" size="1.27" layer="28" ratio="10" rot="MR0"/>
+<element name="R19" library="rcl" library_urn="urn:adsk.eagle:library:334" package="R1206" package3d_urn="urn:adsk.eagle:package:23540/2" value="2k" x="36.6" y="32.5" smashed="yes" rot="MR0">
+<attribute name="NAME" x="39.648" y="34.024" size="1.27" layer="26" ratio="10" rot="MR0"/>
+<attribute name="POPULARITY" value="41" x="36.6" y="32.5" size="1.778" layer="28" rot="MR0" display="off"/>
+<attribute name="SPICEPREFIX" value="R" x="36.6" y="32.5" size="1.778" layer="28" rot="MR0" display="off"/>
+<attribute name="VALUE" x="38.8606" y="31.865" size="1.27" layer="28" ratio="10" rot="MR0"/>
 </element>
 <element name="XS1" library="dragberry" package="CWF-2" value="CWF-2" x="36" y="36" smashed="yes"/>
@@
 </element>
 <element name="SA2" library="dragberry" package="KLS7-6X6" value="BUTTON-TACT-KLS-6X6" x="14.8" y="44" smashed="yes" rot="R90"/>
+<element name="R26" library="rcl" library_urn="urn:adsk.eagle:library:334" package="R1206" package3d_urn="urn:adsk.eagle:package:23540/2" value="" x="31.5" y="33.8" smashed="yes" rot="MR270">
+<attribute name="NAME" x="30.23" y="35.07" size="1.27" layer="26" rot="MR270"/>
+<attribute name="POPULARITY" value="41" x="31.5" y="33.8" size="1.778" layer="28" rot="MR270" display="off"/>
+<attribute name="SPICEPREFIX" value="R" x="31.5" y="33.8" size="1.778" layer="28" rot="MR270" display="off"/>
+<attribute name="VALUE" x="34.04" y="35.07" size="1.27" layer="28" rot="MR270"/>
+</element>
 </elements>
 <signals>
@@
 <wire x1="49.54" y1="29.66" x2="49.54" y2="31" width="1.27" layer="16"/>
 <wire x1="50.87" y1="28.33" x2="49.54" y2="29.66" width="1.27" layer="16"/>
-<wire x1="35.43" y1="27.8" x2="37.13" y2="26.1" width="0.508" layer="16"/>
-<wire x1="45.2" y1="26.1" x2="37.13" y2="26.1" width="0.508" layer="16"/>
+<wire x1="36.33" y1="27.8" x2="38.03" y2="26.1" width="0.508" layer="16"/>
+<wire x1="45.2" y1="26.1" x2="38.03" y2="26.1" width="0.508" layer="16"/>
 <wire x1="45.2" y1="26.1" x2="47.8" y2="23.5" width="0.508" layer="16"/>
 <wire x1="50.87" y1="24.7" x2="50.87" y2="25.3" width="0.508" layer="16"/>
@@
 <wire x1="27.2" y1="34.1" x2="27.2" y2="33.3" width="1.27" layer="16"/>
 <wire x1="33.8" y1="24.4" x2="33" y2="25.2" width="1.27" layer="16"/>
-<wire x1="33" y1="27.5" x2="27.2" y2="33.3" width="1.27" layer="16"/>
+<wire x1="33" y1="27.5" x2="30.7" y2="29.8" width="1.27" layer="16"/>
+<wire x1="30.75" y1="29.75" x2="27.2" y2="33.3" width="1.27" layer="16"/>
 <wire x1="44.89" y1="23.1" x2="43.59" y2="24.4" width="1.27" layer="16"/>
 <wire x1="43.59" y1="24.4" x2="33.8" y2="24.4" width="1.27" layer="16"/>
@@
 <wire x1="93" y1="27.9" x2="91.725" y2="29.175" width="0.508" layer="16"/>
 <wire x1="33" y1="25.2" x2="33" y2="27.2" width="1.27" layer="16"/>
+<contactref element="R26" pad="2"/>
+<wire x1="30.7" y1="29.8" x2="31.5" y2="30.6" width="0.508" layer="16"/>
+<wire x1="31.5" y1="32.378" x2="31.5" y2="30.6" width="0.508" layer="16"/>
 </signal>
 <signal name="N$1">
@@
 <contactref element="VT6" pad="G"/>
 <contactref element="R19" pad="1"/>
-<wire x1="40.070021875" y1="31" x2="38.670021875" y2="32.4" width="0.508" layer="16"/>
-<wire x1="38.670021875" y1="32.4" x2="36.522" y2="32.4" width="0.508" layer="16"/>
-<wire x1="39.87" y1="31" x2="39.87" y2="29.7" width="0.508" layer="16"/>
-<wire x1="37.97" y1="27.8" x2="39.87" y2="29.7" width="0.508" layer="16"/>
-<wire x1="44.46" y1="31" x2="40.070021875" y2="31" width="1.27" layer="16"/>
-<wire x1="40.070021875" y1="31" x2="39.87" y2="31" width="1.27" layer="16"/>
+<wire x1="40.570021875" y1="31" x2="39.070021875" y2="32.5" width="0.508" layer="16"/>
+<wire x1="39.070021875" y1="32.5" x2="38.022" y2="32.5" width="0.508" layer="16"/>
+<wire x1="40.47" y1="31" x2="40.47" y2="29.4" width="0.508" layer="16"/>
+<wire x1="38.87" y1="27.8" x2="40.47" y2="29.4" width="0.508" layer="16"/>
+<wire x1="44.46" y1="31" x2="40.570021875" y2="31" width="1.27" layer="16"/>
+<wire x1="40.570021875" y1="31" x2="40.47" y2="31" width="1.27" layer="16"/>
 </signal>
 <signal name="N$40">
 <contactref element="R18" pad="2"/>
 <contactref element="VT5" pad="2"/>
-<wire x1="36.7" y1="29.705" x2="33.075" y2="29.705" width="0.508" layer="16"/>
-<wire x1="33.075" y1="29.705" x2="28.98" y2="33.8" width="0.508" layer="16"/>
-<wire x1="28.98" y1="33.8" x2="28.98" y2="35.4" width="0.508" layer="16"/>
+<wire x1="33.31995625" y1="30.6561375" x2="34.11153125" y2="29.705" width="0.508" layer="16"/>
+<wire x1="37.6" y1="29.705" x2="34.11153125" y2="29.705" width="0.508" layer="16"/>
+<wire x1="31.5" y1="35.222" x2="31.5" y2="35.14" width="0.508" layer="16"/>
+<wire x1="31.5" y1="35.14" x2="28.98" y2="35.14" width="0.508" layer="16"/>
+<wire x1="28.98" y1="35.14" x2="28.98" y2="35.4" width="0.508" layer="16"/>
+<contactref element="R26" pad="1"/>
+<wire x1="31.5" y1="35.222" x2="32.878" y2="35.222" width="0.508" layer="16"/>
+<wire x1="33.31995625" y1="34.78004375" x2="33.31995625" y2="30.6561375" width="0.508" layer="16"/>
+<wire x1="32.878" y1="35.222" x2="33.31995625" y2="34.78004375" width="0.508" layer="16"/>
 </signal>
 <signal name="N$42">
@@
 <wire x1="34.678" y1="36.072" x2="34.75" y2="36" width="1.27" layer="16"/>
 <wire x1="34.071003125" y1="36.678996875" x2="34.75" y2="36" width="0.508" layer="16"/>
-<wire x1="33.678" y1="32.4" x2="33.678" y2="34.8" width="0.508" layer="16"/>
-<wire x1="34.678" y1="35.8" x2="33.678" y2="34.8" width="0.508" layer="16"/>
-<wire x1="34.678" y1="36.072" x2="34.678" y2="35.8" width="0.508" layer="16"/>
+<wire x1="35.178" y1="32.5" x2="34.678" y2="33" width="0.508" layer="16"/>
+<wire x1="34.678" y1="36.072" x2="34.678" y2="33" width="0.508" layer="16"/>
 <wire x1="33.6" y1="45.5" x2="28.93" y2="45.5" width="1.27" layer="16"/>
 </signal>
@@
 <contactref element="VT6" pad="D"/>
 <contactref element="C7" pad="+"/>
-<wire x1="37.25" y1="36" x2="39.25" y2="34" width="1.27" layer="16"/>
+<wire x1="40.05" y1="34" x2="38.05" y2="36" width="1.27" layer="16"/>
+<wire x1="37.25" y1="36" x2="38.05" y2="36" width="1.27" layer="16"/>
 <wire x1="45.99715" y1="34" x2="47" y2="32.99715" width="1.27" layer="16"/>
 <wire x1="47" y1="32.99715" x2="47" y2="31" width="1.27" layer="16"/>
-<wire x1="39.25" y1="34" x2="45.99715" y2="34" width="1.27" layer="16"/>
+<wire x1="40.05" y1="34" x2="45.99715" y2="34" width="1.27" layer="16"/>
 <wire x1="47" y1="31" x2="47" y2="28.4" width="1.27" layer="16"/>
 <wire x1="48.33" y1="27.07" x2="48.33" y2="25.3" width="1.27" layer="16"/>
