File: boards/pump-board-1.0/pump-board-1.0.sch (EAGLE design)
At the start: 59 parts, among them IC1 74HC595D, IC2 74HC595D, IC3 ATMEGA48/88/168-PU, IC4 7805TV

Commit message: pump code
Parts:
- R18: value (none) -> 510
- R19: value (none) -> 2k
Changed lines of the file:
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@@
 <part name="VT5" library="dragberry" deviceset="2N2222" device="" package3d_urn="urn:adsk.eagle:package:28523/2"/>
 <part name="VT6" library="dragberry" deviceset="IRF1404" device="" package3d_urn="urn:adsk.eagle:package:29490/1"/>
-<part name="R18" library="rcl" library_urn="urn:adsk.eagle:library:334" deviceset="R-EU_" device="0207/10" package3d_urn="urn:adsk.eagle:package:23491/2"/>
-<part name="R19" library="rcl" library_urn="urn:adsk.eagle:library:334" deviceset="R-EU_" device="R1206" package3d_urn="urn:adsk.eagle:package:23540/2"/>
+<part name="R18" library="rcl" library_urn="urn:adsk.eagle:library:334" deviceset="R-EU_" device="0207/10" package3d_urn="urn:adsk.eagle:package:23491/2" value="510"/>
+<part name="R19" library="rcl" library_urn="urn:adsk.eagle:library:334" deviceset="R-EU_" device="R1206" package3d_urn="urn:adsk.eagle:package:23540/2" value="2k"/>
 <part name="GND3" library="supply1" library_urn="urn:adsk.eagle:library:371" deviceset="GND" device=""/>
 <part name="SUPPLY1" library="supply2" library_urn="urn:adsk.eagle:library:372" deviceset="+12V" device=""/>

Commit message: pump
Parts:
- added R26: (no value), rcl:R-EU_R1206
Connections:
- net N$40: now also R26.1
- net VCC: now also R26.2
Changed lines of the file:
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@@
 <part name="C11" library="rcl" deviceset="C-EU" device="C1206" package3d_urn="urn:adsk.eagle:package:23618/2" value="1u"/>
 <part name="SA2" library="dragberry" deviceset="BUTTON" device="-TACT-KLS-6X6"/>
+<part name="R26" library="rcl" library_urn="urn:adsk.eagle:library:334" deviceset="R-EU_" device="R1206" package3d_urn="urn:adsk.eagle:package:23540/2"/>
+<part name="P+4" library="supply1" library_urn="urn:adsk.eagle:library:371" deviceset="VCC" device=""/>
 </parts>
 <sheets>
@@
 <attribute name="NAME" x="-21.59" y="53.34" size="1.778" layer="95"/>
 <attribute name="VALUE" x="-21.59" y="46.99" size="1.778" layer="96"/>
+</instance>
+<instance part="R26" gate="G$1" x="-63.5" y="-63.5" smashed="yes" rot="R90">
+<attribute name="NAME" x="-64.9986" y="-67.31" size="1.778" layer="95" rot="R90"/>
+<attribute name="VALUE" x="-60.198" y="-67.31" size="1.778" layer="96" rot="R90"/>
+</instance>
+<instance part="P+4" gate="VCC" x="-63.5" y="-43.18" smashed="yes">
+<attribute name="VALUE" x="-66.04" y="-45.72" size="1.778" layer="96" rot="R90"/>
 </instance>
 </instances>
@@
 <wire x1="-43.18" y1="63.5" x2="-58.42" y2="63.5" width="0.1524" layer="91"/>
 <junction x="-58.42" y="63.5"/>
+</segment>
+<segment>
+<pinref part="P+4" gate="VCC" pin="VCC"/>
+<pinref part="R26" gate="G$1" pin="2"/>
+<wire x1="-63.5" y1="-45.72" x2="-63.5" y2="-58.42" width="0.1524" layer="91"/>
 </segment>
 </net>
@@
 <pinref part="VT5" gate="G$1" pin="B"/>
 <wire x1="-63.5" y1="-76.2" x2="-60.96" y2="-76.2" width="0.1524" layer="91"/>
-</segment>
-</net>
+<pinref part="R26" gate="G$1" pin="1"/>
+<wire x1="-63.5" y1="-68.58" x2="-63.5" y2="-76.2" width="0.1524" layer="91"/>
+<junction x="-63.5" y="-76.2"/>
+</segment>
+</net>
