File: boards/galvanika-board-2.2-gme12864/galvanika-board-2.2.brd (EAGLE design)
At the start: 250 x 150 mm, 184 parts, among them IC1 LM358D, IC2 LM358D, IC3 LM358D

Commit message: Boards V2.2
Parts:
- removed HG1: WD-G0906WY-BOARD, dragberry:WD-G0906WY-BOARD
- removed JP2: (no value), pinhead:1X04
- added JP1: (no value), pinhead:1X03
- added U$1: DISPLAY-OLED-128X64-I2C, diy-modules:DISPLAY-OLED-128X64-I2C
Connections:
- removed net N$45: DD1.P$6, JP2.3
- removed net N$48: DD1.P$7, JP2.2
- removed net N$49: DD1.P$8, JP2.1
- removed net N$95: DD1.P$16, HG1.P$4
- removed net N$96: DD1.P$17, HG1.P$5
- new net N$77: DD1.P$16, U$1.3
- new net N$80: DD1.P$17, U$1.4
- net BRANCH-CTRL-A: now also DD1.P$9; no longer DD1.P$10
- net BRANCH-CTRL-B: now also DD1.P$8; no longer DD1.P$9
- net GND: now also U$1.1; no longer HG1.P$3, HG1.P$7
- net MODE-CTRL-A: now also DD1.P$12; no longer DD1.P$13
- net MODE-CTRL-B: now also DD1.P$11; no longer DD1.P$12
- net MODE-CTRL-C: now also DD1.P$10; no longer DD1.P$11
- net N$11: now also DD1.P$6, JP1.2; no longer DD1.P$14, HG1.P$1
- net N$2: now also DD1.P$5, JP1.3; no longer DD1.P$15, HG1.P$2
- net N$35: now also DD1.P$7, JP1.1; no longer DD1.P$5, JP2.4
- net VCC: now also U$1.2; no longer HG1.P$10, HG1.P$6, HG1.P$9
Routing:
- net GND: track 2448.4 -> 2371.0 mm
- net N$96: track 59.5 -> 0.00 mm
- net N$95: track 59.2 -> 0.00 mm
- net N$77: track 0.00 -> 57.0 mm
- net N$80: track 0.00 -> 54.0 mm
- net N$2: track 56.0 -> 11.4 mm
- net N$11: track 55.5 -> 11.4 mm
- net ADC0: track 93.2 -> 105.4 mm
- net N$49: track 11.4 -> 0.00 mm
- net N$48: track 11.4 -> 0.00 mm
- net N$45: track 11.4 -> 0.00 mm
- net N$10: track 240.4 -> 230.6 mm
- net BRANCH-CTRL-B: track 153.6 -> 160.3 mm
- net N$9: track 160.8 -> 154.6 mm
- net ADC3: track 216.7 -> 213.3 mm
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Other:
- board text added: "DRAGBERRY 2021.02"
- board text removed: "DRAGBERRY 2021.01"
