File: boards/galvanika-board-2.2-gmg12864/galvanika-board-2.2.brd (EAGLE design)
At the start: 250 x 150 mm, 184 parts, among them IC1 LM358D, IC2 LM358D, IC3 LM358D

Commit message: Boards V2.2
Parts:
- removed HG1: WD-G0906WY-BOARD, dragberry:WD-G0906WY-BOARD
- removed JP2: (no value), pinhead:1X04
- added HG2: GMG1286406D, dragberry:GMG12864
- added JP1: (no value), pinhead:1X03
- moved R44 8.41 mm to (85.8, 40.2)
- moved R87 3.80 mm to (23.4, 45.2), turned to 270 degrees
- moved R17 2.92 mm to (26.6, 39.1), turned to 90 degrees
Connections:
- removed net N$95: DD1.P$16, HG1.P$4
- removed net N$96: DD1.P$17, HG1.P$5
- new net N$77: DD1.P$14, HG2.P$2
- new net N$80: DD1.P$13, HG2.P$1
- net BRANCH-CTRL-A: now also DD1.P$9; no longer DD1.P$10
- net BRANCH-CTRL-B: now also DD1.P$8; no longer DD1.P$9
- net GND: now also HG2.P$7, HG2.P$9; no longer HG1.P$3, HG1.P$7
- net MODE-CTRL-A: now also DD1.P$12; no longer DD1.P$13
- net MODE-CTRL-B: now also DD1.P$11; no longer DD1.P$12
- net MODE-CTRL-C: now also DD1.P$10; no longer DD1.P$11
- net N$11: now also DD1.P$17, HG2.P$5; no longer DD1.P$14, HG1.P$1
- net N$2: now also DD1.P$16, HG2.P$4; no longer DD1.P$15, HG1.P$2
- net N$35: now also JP1.3; no longer JP2.4
- net N$45: now also JP1.2; no longer JP2.3
- net N$48: now also JP1.1; no longer JP2.2
- net N$49: now also DD1.P$15, HG2.P$3; no longer DD1.P$8, JP2.1
- net VCC: now also HG2.P$6, HG2.P$8; no longer HG1.P$10, HG1.P$6, HG1.P$9
Routing:
- net N$96: track 59.5 -> 0.00 mm
- net N$95: track 59.2 -> 0.00 mm
- net N$80: track 0.00 -> 46.7 mm
- net N$77: track 0.00 -> 45.3 mm
- net GND: track 2448.4 -> 2404.8 mm, vias 26 -> 28
- net N$49: track 11.4 -> 42.0 mm
- net ADC0: track 93.2 -> 117.2 mm
- net BRANCH-CTRL-B: track 153.6 -> 132.3 mm, vias 4 -> 6
- net N$11: track 55.5 -> 38.1 mm
- net N$2: track 56.0 -> 40.2 mm
- net MODE-CTRL-A: track 50.8 -> 64.1 mm
- net N$10: track 240.4 -> 228.5 mm
- net N$9: track 160.8 -> 151.9 mm
- net POWER-CTRL-A: track 131.6 -> 125.6 mm
- net VCC: track 836.5 -> 831.3 mm
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Other:
- board text added: "DRAGBERRY 2021.02"
- board text removed: "DRAGBERRY 2021.01"
