File: boards/galvanika-board-2.2-gmg12864/galvanika-board-2.2.sch (EAGLE design)
At the start: 184 parts, among them IC1 LM358D, IC2 LM358D, IC3 LM358D

Commit message: Boards V2.2
Parts:
- removed HG1: WD-G0906WY-BOARD, dragberry:WD-G0906WY-BOARD
- removed JP2: (no value), pinhead:PINHD-1X4
- added HG2: GMG1286406D, dragberry:GMG1286406D
- added JP1: (no value), pinhead:PINHD-1X3
Connections:
- removed net N$95: DD1.PB8, HG1.CS
- removed net N$96: DD1.PB9, HG1.RESET
- new net N$77: DD1.PB6, HG2.RST
- new net N$80: DD1.PB5, HG2.CS
- net BRANCH-CTRL-A: now also DD1.PA12; no longer DD1.PA15
- net BRANCH-CTRL-B: now also DD1.PA11; no longer DD1.PA12
- net GND: now also HG2.GND, HG2.LED-K; no longer HG1.GND, HG1.LED-
- net MODE-CTRL-A: now also DD1.PB4; no longer DD1.PB5
- net MODE-CTRL-B: now also DD1.PB3; no longer DD1.PB4
- net MODE-CTRL-C: now also DD1.PA15; no longer DD1.PB3
- net N$11: now also DD1.PB9, HG2.SDA; no longer DD1.PB6, HG1.CLK
- net N$2: now also DD1.PB8, HG2.SCK; no longer DD1.PB7, HG1.DATA
- net N$35: now also JP1.3; no longer JP2.4
- net N$45: now also JP1.2; no longer JP2.3
- net N$48: now also JP1.1; no longer JP2.2
- net N$49: now also DD1.PB7, HG2.RS; no longer DD1.PA11, JP2.1
- net VCC: now also HG2.LED-A, HG2.VCC; no longer HG1.LED+, HG1.VCC@1, HG1.VCC@2
