File: boards/galvanika-board-2.2-jlx12864g/galvanika-board-2.2.brd (EAGLE design)
At the start: 250 x 150 mm, 184 parts, among them IC1 LM358D, IC2 LM358D, IC3 LM358D

Commit message: Boards V2.2
Connections:
- net BRANCH-CTRL-C: now also DD1.P$4; no longer DD1.P$7
- net N$35: now also DD1.P$5; no longer DD1.P$4
- net N$45: now also DD1.P$6; no longer DD1.P$5
- net N$48: now also DD1.P$7; no longer DD1.P$6
Routing:
- net BRANCH-CTRL-C: track 86.7 -> 82.5 mm
- net N$35: track 12.1 -> 11.5 mm
Changed lines of the file:
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@@
 <wire x1="59" y1="121.9564" x2="58.5" y2="121.4564" width="0.508" layer="16"/>
 <wire x1="58.5" y1="121.4564" x2="58.5" y2="111.5" width="0.508" layer="16"/>
-<wire x1="48.75" y1="101.75" x2="58.5" y2="111.5" width="0.508" layer="16"/>
-<contactref element="DD1" pad="P$7"/>
-<wire x1="48.75" y1="99.9" x2="48.75" y2="101.75" width="0.508" layer="16"/>
-<wire x1="45.88" y1="99.25" x2="48.1" y2="99.25" width="0.508" layer="16"/>
-<wire x1="48.1" y1="99.25" x2="48.75" y2="99.9" width="0.508" layer="16"/>
+<wire x1="54.05" y1="107.05" x2="58.5" y2="111.5" width="0.508" layer="16"/>
+<contactref element="DD1" pad="P$4"/>
+<wire x1="45.88" y1="106.87" x2="53.87" y2="106.87" width="0.508" layer="16"/>
+<wire x1="53.87" y1="106.87" x2="54.05" y2="107.05" width="0.508" layer="16"/>
 </signal>
 <signal name="N$64">
@@
 <wire x1="52.20999375" y1="39.9" x2="52.20999375" y2="42.59000625" width="0.508" layer="16"/>
 </signal>
-<signal name="N$35">
-<contactref element="DD1" pad="P$4"/>
-<wire x1="45.88" y1="106.87" x2="37.25" y2="106.87" width="1.27" layer="16"/>
-<wire x1="37.25" y1="106.87" x2="35.53" y2="106.87" width="1.27" layer="16"/>
-<wire x1="35.56" y1="106.87" x2="37.25" y2="106.87" width="0.2" layer="16"/>
-<contactref element="JP1" pad="3"/>
-<wire x1="35.5" y1="106.84" x2="35.53" y2="106.87" width="1.27" layer="16"/>
-</signal>
-<signal name="N$45">
-<contactref element="DD1" pad="P$5"/>
-<wire x1="45.88" y1="104.33" x2="36.12" y2="104.33" width="1.27" layer="16"/>
-<wire x1="35.56" y1="104.33" x2="36.12" y2="104.33" width="0.2" layer="16"/>
-<contactref element="JP1" pad="2"/>
-<wire x1="35.5" y1="104.3" x2="35.53" y2="104.33" width="1.27" layer="16"/>
-<wire x1="35.53" y1="104.33" x2="36.12" y2="104.33" width="1.27" layer="16"/>
-</signal>
-<signal name="N$48">
-<contactref element="DD1" pad="P$6"/>
-<wire x1="45.88" y1="101.79" x2="36.75" y2="101.79" width="1.27" layer="16"/>
-<wire x1="36.75" y1="101.79" x2="35.53" y2="101.79" width="1.27" layer="16"/>
-<wire x1="35.56" y1="101.79" x2="36.75" y2="101.79" width="0.2" layer="16"/>
-<contactref element="JP1" pad="1"/>
-<wire x1="35.5" y1="101.76" x2="35.53" y2="101.79" width="1.27" layer="16"/>
-</signal>
 <signal name="N$17">
 <contactref element="SA6" pad="P$1"/>
@@
 <wire x1="47.13" y1="44.17" x2="47.13" y2="39.9" width="0.508" layer="16"/>
 </signal>
+<signal name="N$35">
+<contactref element="DD1" pad="P$5"/>
+<contactref element="JP1" pad="3"/>
+<wire x1="45.88" y1="104.33" x2="43.97" y2="104.33" width="1.27" layer="16"/>
+<wire x1="43.97" y1="104.33" x2="41.4" y2="106.9" width="1.27" layer="16"/>
+<wire x1="41.4" y1="106.9" x2="35.56" y2="106.9" width="1.27" layer="16"/>
+<wire x1="35.56" y1="106.9" x2="35.5" y2="106.84" width="1.27" layer="16"/>
+</signal>
+<signal name="N$45">
+<contactref element="JP1" pad="2"/>
+<contactref element="DD1" pad="P$6"/>
+<wire x1="45.88" y1="101.79" x2="42.91" y2="101.79" width="1.27" layer="16"/>
+<wire x1="42.91" y1="101.79" x2="40.4" y2="104.3" width="1.27" layer="16"/>
+<wire x1="40.4" y1="104.3" x2="35.5" y2="104.3" width="1.27" layer="16"/>
+</signal>
+<signal name="N$48">
+<contactref element="JP1" pad="1"/>
+<contactref element="DD1" pad="P$7"/>
+<wire x1="45.88" y1="99.25" x2="41.85" y2="99.25" width="1.27" layer="16"/>
+<wire x1="39.34" y1="101.76" x2="35.5" y2="101.76" width="1.27" layer="16"/>
+<wire x1="41.85" y1="99.25" x2="39.34" y2="101.76" width="1.27" layer="16"/>
+</signal>
 </signals>

Commit message: Galvanika v2.2
Parts:
- moved HG1 0.70 mm to (61.8, 21.0)
Routing:
- net GND: track 2377.8 -> 2380.0 mm
- net N$77: track 46.7 -> 47.6 mm
