File: boards/galvanika-board-2.2-jlx12864g/galvanika-board-2.2.sch (EAGLE design)
At the start: 184 parts, among them IC1 LM358D, IC2 LM358D, IC3 LM358D

Commit message: Boards V2.2
Connections:
- net BRANCH-CTRL-C: now also DD1.PB15; no longer DD1.PA10
- net N$35: now also DD1.PA8; no longer DD1.PB15
- net N$45: now also DD1.PA9; no longer DD1.PA8
- net N$48: now also DD1.PA10; no longer DD1.PA9
Other:
- moved on the sheet: JP1
Changed lines of the file:
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@@
 </instance>
 <instance part="HG1" gate="G$1" x="-279.4" y="-152.4" smashed="yes" rot="R180"/>
-<instance part="JP1" gate="A" x="-238.76" y="-127" smashed="yes" rot="R180">
-<attribute name="NAME" x="-232.41" y="-132.715" size="1.778" layer="95" rot="R180"/>
-<attribute name="VALUE" x="-232.41" y="-119.38" size="1.778" layer="96" rot="R180"/>
+<instance part="JP1" gate="A" x="-238.76" y="-129.54" smashed="yes" rot="R180">
+<attribute name="NAME" x="-232.41" y="-135.255" size="1.778" layer="95" rot="R180"/>
+<attribute name="VALUE" x="-232.41" y="-121.92" size="1.778" layer="96" rot="R180"/>
 </instance>
 </instances>
@@
 </segment>
 <segment>
-<pinref part="DD1" gate="G$1" pin="PA10"/>
-<wire x1="-223.52" y1="-132.08" x2="-218.44" y2="-132.08" width="0.1524" layer="91"/>
+<pinref part="DD1" gate="G$1" pin="PB15"/>
+<wire x1="-223.52" y1="-124.46" x2="-218.44" y2="-124.46" width="0.1524" layer="91"/>
 </segment>
 </net>
@@
 </segment>
 </net>
-<net name="N$35" class="0">
-<segment>
-<pinref part="DD1" gate="G$1" pin="PB15"/>
-<wire x1="-218.44" y1="-124.46" x2="-236.22" y2="-124.46" width="0.1524" layer="91"/>
-<pinref part="JP1" gate="A" pin="3"/>
-</segment>
-</net>
-<net name="N$45" class="0">
-<segment>
-<pinref part="DD1" gate="G$1" pin="PA8"/>
-<wire x1="-218.44" y1="-127" x2="-236.22" y2="-127" width="0.1524" layer="91"/>
-<pinref part="JP1" gate="A" pin="2"/>
-</segment>
-</net>
-<net name="N$48" class="0">
-<segment>
-<pinref part="DD1" gate="G$1" pin="PA9"/>
-<wire x1="-218.44" y1="-129.54" x2="-236.22" y2="-129.54" width="0.1524" layer="91"/>
-<pinref part="JP1" gate="A" pin="1"/>
-</segment>
-</net>
 <net name="N$17" class="0">
 <segment>
@@
 </segment>
 </net>
+<net name="N$35" class="0">
+<segment>
+<pinref part="DD1" gate="G$1" pin="PA8"/>
+<pinref part="JP1" gate="A" pin="3"/>
+<wire x1="-218.44" y1="-127" x2="-236.22" y2="-127" width="0.1524" layer="91"/>
+</segment>
+</net>
+<net name="N$45" class="0">
+<segment>
+<pinref part="JP1" gate="A" pin="2"/>
+<pinref part="DD1" gate="G$1" pin="PA9"/>
+<wire x1="-236.22" y1="-129.54" x2="-218.44" y2="-129.54" width="0.1524" layer="91"/>
+</segment>
+</net>
+<net name="N$48" class="0">
+<segment>
+<pinref part="JP1" gate="A" pin="1"/>
+<pinref part="DD1" gate="G$1" pin="PA10"/>
+<wire x1="-236.22" y1="-132.08" x2="-218.44" y2="-132.08" width="0.1524" layer="91"/>
+</segment>
+</net>
